File: midi_dac.sch (KiCad schematic (older format))
At the start: 67 parts, among them CON1 SN49B12B, J10 USB_A, J11 Conn_02x05_Odd_Even, J12 Conn_01x03_Male, J13 Conn_01x04_Male, J9 Conn_01x05_Male, SW4 SW_Push_Dual, SW5 SW_Push_Dual, SW6 SW_Push_Dual, U5 STM32F407VGT6, U6 PCM5102, U7 STMPS2141STR

Commit message: Make most changes for final design
Parts:
- added C?: 100nF, symbol Device:C_Small
- added U?: USBLC6-2SC6, Package_TO_SOT_SMD:SOT-23-6, symbol Power_Protection:USBLC6-2SC6
- D4: value LED -> ORA_LED
- D5: value LED -> RED_LED
Connections:
- net labels added: +5V, USB_DM, USB_DP
- wire segments 297 -> 307
Other:
- note added: "USB ESD Protection"
- moved on the sheet: D2, D3, D4, D5, R25, R26, R27, R28

Commit message: Update power supply system
Parts:
- gave numbers to parts that had none: 2
Changed lines of the file:
@@
 	1    0    0    -1
 $EndComp
-$Comp
-L power:+3.3V #PWR085
-U 1 1 609ED1C8
-P 9100 1150
-F 0 "#PWR085" H 9100 1000 50  0001 C CNN
-F 1 "+3.3V" H 8950 1200 50  0000 C CNN
-F 2 "" H 9100 1150 50  0001 C CNN
-F 3 "" H 9100 1150 50  0001 C CNN
-	1    9100 1150
-	1    0    0    -1
-$EndComp
-Wire Wire Line
-	9100 1150 9100 1200
 Wire Wire Line
 	9100 1400 9250 1400
@@
 Connection ~ 2250 7400
 $Comp
-L power:+3.3V #PWR096
-U 1 1 61B6F7C5
-P 10300 850
-F 0 "#PWR096" H 10300 700 50  0001 C CNN
-F 1 "+3.3V" H 10315 1023 50  0000 C CNN
-F 2 "" H 10300 850 50  0001 C CNN
-F 3 "" H 10300 850 50  0001 C CNN
-	1    10300 850
-	1    0    0    -1
-$EndComp
-$Comp
 L power:GND #PWR097
 U 1 1 61B6FB7D
@@
 $EndComp
 $Comp
-L power:+3.3V #PWR?
+L power:+3.3V #PWR018
 U 1 1 605E8F70
 P 2250 7100
-F 0 "#PWR?" H 2250 6950 50  0001 C CNN
+F 0 "#PWR018" H 2250 6950 50  0001 C CNN
 F 1 "+3.3V" H 2265 7273 50  0000 C CNN
 F 2 "" H 2250 7100 50  0001 C CNN
@@
 Connection ~ 2250 7150
 $Comp
-L Power_Protection:USBLC6-2SC6 U?
+L Power_Protection:USBLC6-2SC6 U9
 U 1 1 60608657
 P 5050 5600
-F 0 "U?" H 5200 6050 50  0000 C CNN
+F 0 "U9" H 5200 6050 50  0000 C CNN
 F 1 "USBLC6-2SC6" H 5400 5950 50  0000 C CNN
 F 2 "Package_TO_SOT_SMD:SOT-23-6" H 4300 6000 50  0001 C CNN
@@
 $EndComp
 $Comp
-L power:+5V #PWR?
+L power:+5V #PWR057
 U 1 1 606180F0
 P 5050 5050
-F 0 "#PWR?" H 5050 4900 50  0001 C CNN
+F 0 "#PWR057" H 5050 4900 50  0001 C CNN
 F 1 "+5V" H 5065 5223 50  0000 C CNN
 F 2 "" H 5050 5050 50  0001 C CNN
@@
 	5050 5050 5050 5100
 $Comp
-L power:GND #PWR?
+L power:GND #PWR098
 U 1 1 606342CD
 P 5050 6150
-F 0 "#PWR?" H 5050 5900 50  0001 C CNN
+F 0 "#PWR098" H 5050 5900 50  0001 C CNN
 F 1 "GND" H 5055 5977 50  0000 C CNN
 F 2 "" H 5050 6150 50  0001 C CNN
@@
 	5050 6150 5050 6100
 $Comp
-L Device:C_Small C?
+L Device:C_Small C57
 U 1 1 6065009D
 P 5550 6100
-F 0 "C?" H 5642 6146 50  0000 L CNN
+F 0 "C57" H 5642 6146 50  0000 L CNN
 F 1 "100nF" H 5642 6055 50  0000 L CNN
 F 2 "" H 5550 6100 50  0001 C CNN
@@
 $EndComp
 $Comp
-L power:+5V #PWR?
+L power:+5V #PWR099
 U 1 1 6065220C
 P 5550 5950
-F 0 "#PWR?" H 5550 5800 50  0001 C CNN
+F 0 "#PWR099" H 5550 5800 50  0001 C CNN
 F 1 "+5V" H 5565 6123 50  0000 C CNN
 F 2 "" H 5550 5950 50  0001 C CNN
@@
 	5550 5950 5550 6000
 $Comp
-L power:GND #PWR?
+L power:GND #PWR0100
 U 1 1 6069ADB3
 P 5550 6250
-F 0 "#PWR?" H 5550 6000 50  0001 C CNN
+F 0 "#PWR0100" H 5550 6000 50  0001 C CNN
 F 1 "GND" H 5555 6077 50  0000 C CNN
 F 2 "" H 5550 6250 50  0001 C CNN
@@
 Text Notes 4000 4800 0    50   ~ 0
 USB ESD Protection
+$Comp
+L power:+5V #PWR085
+U 1 1 609E8B3B
+P 9100 1150
+F 0 "#PWR085" H 9100 1000 50  0001 C CNN
+F 1 "+5V" H 9115 1323 50  0000 C CNN
+F 2 "" H 9100 1150 50  0001 C CNN
+F 3 "" H 9100 1150 50  0001 C CNN
+	1    9100 1150
+	1    0    0    -1
+$EndComp
+Wire Wire Line
+	9100 1150 9100 1200
+$Comp
+L power:+5V #PWR096
+U 1 1 60A20880
+P 10300 850
+F 0 "#PWR096" H 10300 700 50  0001 C CNN
+F 1 "+5V" H 10315 1023 50  0000 C CNN
+F 2 "" H 10300 850 50  0001 C CNN
+F 3 "" H 10300 850 50  0001 C CNN
+	1    10300 850
+	1    0    0    -1
+$EndComp
 $EndSCHEMATC

Commit message: Final iteration before pcb design review
Parts:
- removed HSE2: 8MHz, symbol Device:Crystal_GND23_Small
- added R52: 8k, Resistor_SMD:R_0603_1608Metric, symbol Device:R_Small
- added Y2: 8MHz, Crystal:Crystal_SMD_Abracon_ABM10-4Pin_2.5x2.0mm, symbol Device:Crystal_GND24_Small
- C20, C21, C22, C23, C24, C25, C26, C27, C29, C31, C32, C34, C36, C37, C40, C44, C45, C46, C47, C57: footprint (none) -> Capacitor_SMD:C_0805_2012Metric
- C28, C30, C33, C35, C38, C39, C41, C42, C43: footprint (none) -> Capacitor_SMD:C_0603_1608Metric
- CON1: symbol DIGIKEY_AUDIO_JACK:SN49B12B -> digidraw-rescue:SN49B12B-DIGIKEY_AUDIO_JACK
- D2, D3, D4, D5: footprint (none) -> LED_SMD:LED_0603_1608Metric
- J10, J11: footprint (none) -> Connector_USB:USB_A_Molex_67643_Horizontal
- J12, J13: footprint (none) -> Connector_PinHeader_2.54mm:PinHeader_1x06_P2.54mm_Vertical
- J9: footprint (none) -> Connector_PinHeader_2.54mm:PinHeader_1x08_P2.54mm_Vertical
- R25: value 50 -> 75; footprint (none) -> Resistor_SMD:R_0603_1608Metric
- R26: value 60 -> 75; footprint (none) -> Resistor_SMD:R_0603_1608Metric
- R27: value 65 -> 75; footprint (none) -> Resistor_SMD:R_0603_1608Metric
- R28: value 67.5 -> 75; footprint (none) -> Resistor_SMD:R_0603_1608Metric
- R29, R30, R31, R32, R33, R34, R35, R36, R38, R39, R40, R41, R42, R43, R44, R45, R46: footprint (none) -> Resistor_SMD:R_0603_1608Metric
- R37: value 10k -> 5k; footprint (none) -> Resistor_SMD:R_0603_1608Metric
- SW4, SW5, SW6: footprint (none) -> Button_Switch_SMD:SW_SPST_EVPBF
- U7: symbol DIGIKEY_POWER_SWITCH:STMPS2141STR -> digidraw-rescue:STMPS2141STR-DIGIKEY_POWER_SWITCH
Connections:
- wire segments 307 -> 310

Commit message: Finish schematic
Parts:
- C20, C21, C22, C23, C24, C25, C26, C27, C28, C29, C30, C31, C32, C33, C34, C35, C36, C37, C38, C39, C40, C41, C42, C43, C45, C46: Min Voltage Rating (none) -> 3.3 V
- C44, C47, C57: Min Voltage Rating (none) -> 5.2 V
- D2, D3, D4, D5: Description (none) -> Debug LED
- J10: Description (none) -> Connector for USB Midi
- J11: Description (none) -> STLink Header for programming/debug
- J12: Description (none) -> Header for analog out probes
- J13: Description (none) -> Header for UART Debug
- J9: Description (none) -> Header for I2S Debug
- SW4, SW5, SW6: Description (none) -> Pushbuttons for NRST/BOOT
- U5: Description (none) -> F4 processor for DAC/MIDI subsystem
- U6: Description (none) -> DAC for output
- U9: Description (none) -> USB Micro B ESD protection
- Y2: Description (none) -> HSE crystals
Changed lines of the file:
@@
 F 2 "Package_QFP:LQFP-100_14x14mm_P0.5mm" H 1650 1050 50  0001 R CNN
 F 3 "http://www.st.com/st-web-ui/static/active/en/resource/technical/document/datasheet/DM00037051.pdf" H 2350 3650 50  0001 C CNN
+F 4 "F4 processor for DAC/MIDI subsystem" H 2350 3650 50  0001 C CNN "Description"
 	1    2350 3650
 	1    0    0    -1
@@
 F 2 "Capacitor_SMD:C_0805_2012Metric" H 6300 2650 50  0001 C CNN
 F 3 "~" H 6300 2650 50  0001 C CNN
+F 4 "3.3 V" H 6300 2650 50  0001 C CNN "Min Voltage Rating"
 	1    6300 2650
 	1    0    0    -1
@@
 F 2 "Capacitor_SMD:C_0805_2012Metric" H 6650 2650 50  0001 C CNN
 F 3 "~" H 6650 2650 50  0001 C CNN
+F 4 "3.3 V" H 6650 2650 50  0001 C CNN "Min Voltage Rating"
 	1    6650 2650
 	1    0    0    -1
@@
 F 2 "Capacitor_SMD:C_0805_2012Metric" H 7000 2650 50  0001 C CNN
 F 3 "~" H 7000 2650 50  0001 C CNN
+F 4 "3.3 V" H 7000 2650 50  0001 C CNN "Min Voltage Rating"
 	1    7000 2650
 	1    0    0    -1
@@
 F 2 "Capacitor_SMD:C_0805_2012Metric" H 7350 2650 50  0001 C CNN
 F 3 "~" H 7350 2650 50  0001 C CNN
+F 4 "3.3 V" H 7350 2650 50  0001 C CNN "Min Voltage Rating"
 	1    7350 2650
 	1    0    0    -1
@@
 F 2 "Capacitor_SMD:C_0805_2012Metric" H 7700 2650 50  0001 C CNN
 F 3 "~" H 7700 2650 50  0001 C CNN
+F 4 "3.3 V" H 7700 2650 50  0001 C CNN "Min Voltage Rating"
 	1    7700 2650
 	1    0    0    -1
@@
 F 2 "Capacitor_SMD:C_0805_2012Metric" H 8050 2650 50  0001 C CNN
 F 3 "~" H 8050 2650 50  0001 C CNN
+F 4 "3.3 V" H 8050 2650 50  0001 C CNN "Min Voltage Rating"
 	1    8050 2650
 	1    0    0    -1
@@
 F 2 "Capacitor_SMD:C_0805_2012Metric" H 8400 2650 50  0001 C CNN
 F 3 "~" H 8400 2650 50  0001 C CNN
+F 4 "3.3 V" H 8400 2650 50  0001 C CNN "Min Voltage Rating"
 	1    8400 2650
 	1    0    0    -1
@@
 F 2 "Capacitor_SMD:C_0603_1608Metric" H 8750 2650 50  0001 C CNN
 F 3 "~" H 8750 2650 50  0001 C CNN
+F 4 "3.3 V" H 8750 2650 50  0001 C CNN "Min Voltage Rating"
 	1    8750 2650
 	1    0    0    -1
@@
 F 2 "Capacitor_SMD:C_0805_2012Metric" H 9100 2600 50  0001 C CNN
 F 3 "~" H 9100 2600 50  0001 C CNN
+F 4 "3.3 V" H 9100 2600 50  0001 C CNN "Min Voltage Rating"
 	1    9100 2600
 	1    0    0    -1
@@
 F 2 "Capacitor_SMD:C_0603_1608Metric" H 9500 2600 50  0001 C CNN
 F 3 "~" H 9500 2600 50  0001 C CNN
+F 4 "3.3 V" H 9500 2600 50  0001 C CNN "Min Voltage Rating"
 	1    9500 2600
 	1    0    0    -1
@@
 F 2 "Capacitor_SMD:C_0805_2012Metric" H 550 2100 50  0001 C CNN
 F 3 "~" H 550 2100 50  0001 C CNN
+F 4 "3.3 V" H 550 2100 50  0001 C CNN "Min Voltage Rating"
 	1    550  2100
 	1    0    0    -1
@@
 F 2 "Capacitor_SMD:C_0805_2012Metric" H 950 2100 50  0001 C CNN
 F 3 "~" H 950 2100 50  0001 C CNN
+F 4 "3.3 V" H 950 2100 50  0001 C CNN "Min Voltage Rating"
 	1    950  2100
 	1    0    0    -1
@@
 F 2 "Capacitor_SMD:C_0603_1608Metric" H 7550 1200 50  0001 C CNN
 F 3 "~" H 7550 1200 50  0001 C CNN
+F 4 "3.3 V" H 7550 1200 50  0001 C CNN "Min Voltage Rating"
 	1    7550 1200
 	1    0    0    -1
@@
 F 2 "Capacitor_SMD:C_0603_1608Metric" H 7100 1200 50  0001 C CNN
 F 3 "~" H 7100 1200 50  0001 C CNN
+F 4 "3.3 V" H 7100 1200 50  0001 C CNN "Min Voltage Rating"
 	1    7100 1200
 	1    0    0    -1
@@
 F 2 "Package_SO:TSSOP-20_4.4x6.5mm_P0.65mm" H 7700 6150 50  0001 C CNN
 F 3 "http://www.ti.com/lit/ds/symlink/pcm5102.pdf" H 7700 6150 50  0001 C CNN
+F 4 "DAC for output" H 7750 5400 50  0001 C CNN "Description"
 	1    7750 5400
 	1    0    0    -1
@@
 F 2 "Capacitor_SMD:C_0603_1608Metric" H 9900 5450 50  0001 C CNN
 F 3 "~" H 9900 5450 50  0001 C CNN
+F 4 "3.3 V" H 9900 5450 50  0001 C CNN "Min Voltage Rating"
 	1    9900 5450
 	1    0    0    -1
@@
 F 2 "Capacitor_SMD:C_0603_1608Metric" H 8350 5450 50  0001 C CNN
 F 3 "~" H 8350 5450 50  0001 C CNN
+F 4 "3.3 V" H 8350 5450 50  0001 C CNN "Min Voltage Rating"
 	1    8350 5450
 	1    0    0    -1
@@
 F 2 "Capacitor_SMD:C_0805_2012Metric" H 10200 5800 50  0001 C CNN
 F 3 "~" H 10200 5800 50  0001 C CNN
+F 4 "3.3 V" H 10200 5800 50  0001 C CNN "Min Voltage Rating"
 	1    10200 5800
 	1    0    0    -1
@@
 F 2 "Capacitor_SMD:C_0603_1608Metric" H 9100 5350 50  0001 C CNN
 F 3 "~" H 9100 5350 50  0001 C CNN
+F 4 "3.3 V" H 9100 5350 50  0001 C CNN "Min Voltage Rating"
 	1    9100 5350
 	1    0    0    -1
@@
 F 2 "Capacitor_SMD:C_0603_1608Metric" H 9100 5650 50  0001 C CNN
 F 3 "~" H 9100 5650 50  0001 C CNN
+F 4 "3.3 V" H 9100 5650 50  0001 C CNN "Min Voltage Rating"
 	1    9100 5650
 	1    0    0    -1
@@
 F 2 "Capacitor_SMD:C_0805_2012Metric" H 8750 4000 50  0001 C CNN
 F 3 "~" H 8750 4000 50  0001 C CNN
+F 4 "3.3 V" H 8750 4000 50  0001 C CNN "Min Voltage Rating"
 	1    8750 4000
 	1    0    0    -1
@@
 F 2 "Capacitor_SMD:C_0805_2012Metric" H 10000 4000 50  0001 C CNN
 F 3 "~" H 10000 4000 50  0001 C CNN
+F 4 "3.3 V" H 10000 4000 50  0001 C CNN "Min Voltage Rating"
 	1    10000 4000
 	1    0    0    -1
@@
 F 2 "Capacitor_SMD:C_0805_2012Metric" H 9400 4350 50  0001 C CNN
 F 3 "~" H 9400 4350 50  0001 C CNN
+F 4 "3.3 V" H 9400 4350 50  0001 C CNN "Min Voltage Rating"
 	1    9400 4350
 	-1   0    0    1
@@
 F 2 "Capacitor_SMD:C_0603_1608Metric" H 9600 4350 50  0001 C CNN
 F 3 "~" H 9600 4350 50  0001 C CNN
+F 4 "3.3 V" H 9600 4350 50  0001 C CNN "Min Voltage Rating"
 	1    9600 4350
 	-1   0    0    1
@@
 F 2 "Connector_PinHeader_2.54mm:PinHeader_1x06_P2.54mm_Vertical" H 6350 1200 50  0001 C CNN
 F 3 "~" H 6350 1200 50  0001 C CNN
+F 4 "Header for UART Debug" H 6350 1200 50  0001 C CNN "Description"
 	1    6350 1200
 	-1   0    0    1
@@
 F 2 "Connector_USB:USB_A_Molex_67643_Horizontal" H 5200 2350 50  0001 C CNN
 F 3 " ~" H 5200 2350 50  0001 C CNN
+F 4 "Connector for USB Midi" H 5050 2400 50  0001 C CNN "Description"
 	1    5050 2400
 	1    0    0    -1
@@
 F 2 "Connector_USB:USB_A_Molex_67643_Horizontal" H 5100 4250 50  0001 C CNN
 F 3 "~" H 5100 4250 50  0001 C CNN
+F 4 "STLink Header for programming/debug" H 5100 4250 50  0001 C CNN "Description"
 	1    5100 4250
 	1    0    0    -1
@@
 F 2 "Button_Switch_SMD:SW_SPST_EVPBF" H 3700 7250 50  0001 C CNN
 F 3 "~" H 3700 7250 50  0001 C CNN
+F 4 "Pushbuttons for NRST/BOOT" H 3700 7050 50  0001 C CNN "Description"
 	1    3700 7050
 	1    0    0    -1
@@
 F 2 "Capacitor_SMD:C_0805_2012Metric" H 3700 7400 50  0001 C CNN
 F 3 "~" H 3700 7400 50  0001 C CNN
+F 4 "3.3 V" H 3700 7400 50  0001 C CNN "Min Voltage Rating"
 	1    3700 7400
 	0    -1   -1   0
@@
 F 2 "Connector_PinHeader_2.54mm:PinHeader_1x06_P2.54mm_Vertical" H 5500 1100 50  0001 C CNN
 F 3 "~" H 5500 1100 50  0001 C CNN
+F 4 "Header for analog out probes" H 5500 1100 50  0001 C CNN "Description"
 	1    5500 1100
 	-1   0    0    1
@@
 F 2 "Connector_PinHeader_2.54mm:PinHeader_1x08_P2.54mm_Vertical" H 4600 1100 50  0001 C CNN
 F 3 "~" H 4600 1100 50  0001 C CNN
+F 4 "Header for I2S Debug" H 4600 1100 50  0001 C CNN "Description"
 	1    4600 1100
 	-1   0    0    1
@@
 F 2 "Capacitor_SMD:C_0805_2012Metric" H 10100 1600 50  0001 C CNN
 F 3 "~" H 10100 1600 50  0001 C CNN
+F 4 "5.2 V" H 10100 1600 50  0001 C CNN "Min Voltage Rating"
 	1    10100 1600
 	1    0    0    -1
@@
 F 2 "LED_SMD:LED_0603_1608Metric" H 1600 7400 50  0001 C CNN
 F 3 "~" H 1600 7400 50  0001 C CNN
+F 4 "Debug LED" H 1600 7400 50  0001 C CNN "Description"
 	1    1600 7400
 	1    0    0    1
@@
 F 2 "LED_SMD:LED_0603_1608Metric" H 1600 7650 50  0001 C CNN
 F 3 "~" H 1600 7650 50  0001 C CNN
+F 4 "Debug LED" H 1600 7650 50  0001 C CNN "Description"
 	1    1600 7650
 	1    0    0    1
@@
 F 2 "LED_SMD:LED_0603_1608Metric" H 1600 7900 50  0001 C CNN
 F 3 "~" H 1600 7900 50  0001 C CNN
+F 4 "Debug LED" H 1600 7900 50  0001 C CNN "Description"
 	1    1600 7900
 	1    0    0    1
@@
 F 2 "Capacitor_SMD:C_0805_2012Metric" H 10300 1000 50  0001 C CNN
 F 3 "~" H 10300 1000 50  0001 C CNN
+F 4 "5.2 V" H 10300 1000 50  0001 C CNN "Min Voltage Rating"
 	1    10300 1000
 	1    0    0    -1
@@
 F 2 "Button_Switch_SMD:SW_SPST_EVPBF" H 4900 7250 50  0001 C CNN
 F 3 "~" H 4900 7250 50  0001 C CNN
+F 4 "Pushbuttons for NRST/BOOT" H 4900 7050 50  0001 C CNN "Description"
 	1    4900 7050
 	0    1    1    0
@@
 F 2 "Capacitor_SMD:C_0805_2012Metric" H 4550 7100 50  0001 C CNN
 F 3 "~" H 4550 7100 50  0001 C CNN
+F 4 "3.3 V" H 4550 7100 50  0001 C CNN "Min Voltage Rating"
 	1    4550 7100
 	1    0    0    -1
@@
 F 2 "Button_Switch_SMD:SW_SPST_EVPBF" H 5850 7250 50  0001 C CNN
 F 3 "~" H 5850 7250 50  0001 C CNN
+F 4 "Pushbuttons for NRST/BOOT" H 5850 7050 50  0001 C CNN "Description"
 	1    5850 7050
 	0    1    1    0
@@
 F 2 "Capacitor_SMD:C_0805_2012Metric" H 5500 7100 50  0001 C CNN
 F 3 "~" H 5500 7100 50  0001 C CNN
+F 4 "3.3 V" H 5500 7100 50  0001 C CNN "Min Voltage Rating"
 	1    5500 7100
 	1    0    0    -1
@@
 F 2 "LED_SMD:LED_0603_1608Metric" H 1600 7150 50  0001 C CNN
 F 3 "~" H 1600 7150 50  0001 C CNN
+F 4 "Debug LED" H 1600 7150 50  0001 C CNN "Description"
 	1    1600 7150
 	1    0    0    1
@@
 F 2 "Package_TO_SOT_SMD:SOT-23-6" H 4300 6000 50  0001 C CNN
 F 3 "http://www2.st.com/resource/en/datasheet/CD00050750.pdf" H 5250 5950 50  0001 C CNN
+F 4 "USB Micro B ESD protection" H 5050 5600 50  0001 C CNN "Description"
 	1    5050 5600
 	1    0    0    -1
@@
 F 2 "Capacitor_SMD:C_0805_2012Metric" H 5550 6100 50  0001 C CNN
 F 3 "~" H 5550 6100 50  0001 C CNN
+F 4 "5.2 V" H 5550 6100 50  0001 C CNN "Min Voltage Rating"
 	1    5550 6100
 	1    0    0    -1
@@
 F 2 "Crystal:Crystal_SMD_Abracon_ABM10-4Pin_2.5x2.0mm" H 7300 1000 50  0001 C CNN
 F 3 "~" H 7300 1000 50  0001 C CNN
+F 4 "HSE crystals" H 7300 1000 50  0001 C CNN "Description"
 	1    7300 1000
 	1    0    0    -1

Commit message: Work on pcb layout
Parts:
- J11: footprint Connector_USB:USB_A_Molex_67643_Horizontal -> Connector_PinHeader_2.54mm:PinHeader_2x05_P2.54mm_Vertical
- J12: footprint Connector_PinHeader_2.54mm:PinHeader_1x06_P2.54mm_Vertical -> Connector_PinHeader_2.54mm:PinHeader_1x03_P2.54mm_Vertical
- J13: footprint Connector_PinHeader_2.54mm:PinHeader_1x06_P2.54mm_Vertical -> Connector_PinHeader_2.54mm:PinHeader_1x04_P2.54mm_Vertical
- J9: footprint Connector_PinHeader_2.54mm:PinHeader_1x08_P2.54mm_Vertical -> Connector_PinSocket_2.54mm:PinSocket_1x05_P2.54mm_Vertical
Changed lines of the file:
@@
 F 0 "J13" H 6450 900 50  0000 R CNN
 F 1 "Conn_01x04_Male" V 6300 1450 50  0000 R CNN
-F 2 "Connector_PinHeader_2.54mm:PinHeader_1x06_P2.54mm_Vertical" H 6350 1200 50  0001 C CNN
+F 2 "Connector_PinHeader_2.54mm:PinHeader_1x04_P2.54mm_Vertical" H 6350 1200 50  0001 C CNN
 F 3 "~" H 6350 1200 50  0001 C CNN
 F 4 "Header for UART Debug" H 6350 1200 50  0001 C CNN "Description"
@@
 F 0 "J11" H 5150 4550 50  0000 C CNN
 F 1 "Conn_02x05_Odd_Even" H 5350 3950 50  0000 C CNN
-F 2 "Connector_USB:USB_A_Molex_67643_Horizontal" H 5100 4250 50  0001 C CNN
+F 2 "Connector_PinHeader_2.54mm:PinHeader_2x05_P2.54mm_Vertical" H 5100 4250 50  0001 C CNN
 F 3 "~" H 5100 4250 50  0001 C CNN
 F 4 "STLink Header for programming/debug" H 5100 4250 50  0001 C CNN "Description"
@@
 F 0 "J12" H 5750 900 50  0000 R CNN
 F 1 "Conn_01x03_Male" H 5850 1400 50  0000 R CNN
-F 2 "Connector_PinHeader_2.54mm:PinHeader_1x06_P2.54mm_Vertical" H 5500 1100 50  0001 C CNN
+F 2 "Connector_PinHeader_2.54mm:PinHeader_1x03_P2.54mm_Vertical" H 5500 1100 50  0001 C CNN
 F 3 "~" H 5500 1100 50  0001 C CNN
 F 4 "Header for analog out probes" H 5500 1100 50  0001 C CNN "Description"
@@
 F 0 "J9" H 4700 800 50  0000 R CNN
 F 1 "Conn_01x05_Male" V 4550 1400 50  0000 R CNN
-F 2 "Connector_PinHeader_2.54mm:PinHeader_1x08_P2.54mm_Vertical" H 4600 1100 50  0001 C CNN
+F 2 "Connector_PinSocket_2.54mm:PinSocket_1x05_P2.54mm_Vertical" H 4600 1100 50  0001 C CNN
 F 3 "~" H 4600 1100 50  0001 C CNN
 F 4 "Header for I2S Debug" H 4600 1100 50  0001 C CNN "Description"

Commit message: Decent layout at first glance
Connections:
- net +3.3VADC renamed +3.3VDAC
Changed lines of the file:
@@
 Wire Wire Line
 	7200 5200 7250 5200
-$Comp
-L power:+3.3VADC #PWR092
-U 1 1 6134A6E5
-P 9600 4150
-F 0 "#PWR092" H 9750 4100 50  0001 C CNN
-F 1 "+3.3VADC" H 9500 4250 50  0000 C CNN
-F 2 "" H 9600 4150 50  0001 C CNN
-F 3 "" H 9600 4150 50  0001 C CNN
-	1    9600 4150
-	1    0    0    -1
-$EndComp
 Wire Wire Line
 	9600 4150 9600 4200
 Connection ~ 9600 4200
-$Comp
-L power:+3.3VADC #PWR083
-U 1 1 6135ED8F
-P 7850 4700
-F 0 "#PWR083" H 8000 4650 50  0001 C CNN
-F 1 "+3.3VADC" H 8000 4800 50  0000 C CNN
-F 2 "" H 7850 4700 50  0001 C CNN
-F 3 "" H 7850 4700 50  0001 C CNN
-	1    7850 4700
-	1    0    0    -1
-$EndComp
 $Comp
 L power:GND #PWR082
@@
 Wire Wire Line
 	7300 850  7300 900
+$Comp
+L power:+3.3VDAC #PWR0102
+U 1 1 607DB7E8
+P 7850 4700
+F 0 "#PWR0102" H 8000 4650 50  0001 C CNN
+F 1 "+3.3VDAC" H 7870 4843 50  0000 C CNN
+F 2 "" H 7850 4700 50  0001 C CNN
+F 3 "" H 7850 4700 50  0001 C CNN
+	1    7850 4700
+	1    0    0    -1
+$EndComp
+$Comp
+L power:+3.3VDAC #PWR?
+U 1 1 607E677E
+P 9600 4150
+F 0 "#PWR?" H 9750 4100 50  0001 C CNN
+F 1 "+3.3VDAC" H 9620 4293 50  0000 C CNN
+F 2 "" H 9600 4150 50  0001 C CNN
+F 3 "" H 9600 4150 50  0001 C CNN
+	1    9600 4150
+	1    0    0    -1
+$EndComp
 $EndSCHEMATC

Commit message: Replace components
Parts:
- J9: footprint Connector_PinSocket_2.54mm:PinSocket_1x05_P2.54mm_Vertical -> Connector_PinHeader_2.54mm:PinHeader_1x05_P2.54mm_Vertical
Connections:
- net GPIO_EXTI0 is gone; now on net UART4_TX: U5.23 (PA0)
- net I2S_CK: now also J9.4 (Pin_4); no longer J9.3 (Pin_3)
- net I2S_SD: now also J9.3 (Pin_3); no longer J9.2 (Pin_2)
- net I2S_WS: now also J9.2 (Pin_2); no longer J9.4 (Pin_4)
- net SPI_INT: now also U5.31 (PA6); no longer U5.90 (PB4)
- net UART4_TX: no longer U5.78 (PC10)
- net USB_VBUS_EN: now also U5.69 (PA10); no longer U5.15 (PC0)
- net at U5.18 (PC3): no longer R31.2
- net at U5.54 (PB15): now also R31.2
- no-connect marks 59 -> 60
Other:
- moved on the sheet: R31
Changed lines of the file:
@@
 Wire Wire Line
 	9600 4550 10000 4550
-Text Label 3650 4950 0    50   ~ 0
+Text Label 3650 4450 0    50   ~ 0
 I2S_SD
 Wire Wire Line
-	3400 4950 3250 4950
+	3400 4450 3250 4450
 Wire Notes Line
 	8250 4800 10500 4800
@@
 Wire Wire Line
 	3400 1350 3250 1350
-Text Label 3350 5650 0    50   ~ 0
+Text Label 3400 1250 0    50   ~ 0
 UART4_TX
-Wire Wire Line
-	3350 5650 3250 5650
 $Comp
 L Connector:Conn_01x04_Male J13
@@
 Wire Wire Line
 	3400 2150 3250 2150
-Text Label 3400 4650 0    50   ~ 0
+Text Label 3400 2250 0    50   ~ 0
 USB_VBUS_EN
 Wire Wire Line
-	3400 4650 3250 4650
+	3400 2250 3250 2250
 $Comp
 L digidraw-rescue:STMPS2141STR-DIGIKEY_POWER_SWITCH U7
@@
 Text Label 7200 5100 2    50   ~ 0
 I2S_SD
-Text Label 3400 1250 0    50   ~ 0
-GPIO_EXTI0
 Wire Wire Line
 	3400 1250 3250 1250
@@
 NoConn ~ 3250 1450
 NoConn ~ 3250 1550
-NoConn ~ 3250 1850
 NoConn ~ 3250 2050
-NoConn ~ 3250 2250
+NoConn ~ 3250 4650
 NoConn ~ 3250 2750
 NoConn ~ 3250 2950
@@
 NoConn ~ 3250 4250
 NoConn ~ 3250 4350
-NoConn ~ 3250 4450
 NoConn ~ 3250 4750
 NoConn ~ 3250 4850
@@
 F 0 "J9" H 4700 800 50  0000 R CNN
 F 1 "Conn_01x05_Male" V 4550 1400 50  0000 R CNN
-F 2 "Connector_PinSocket_2.54mm:PinSocket_1x05_P2.54mm_Vertical" H 4600 1100 50  0001 C CNN
+F 2 "Connector_PinHeader_2.54mm:PinHeader_1x05_P2.54mm_Vertical" H 4600 1100 50  0001 C CNN
 F 3 "~" H 4600 1100 50  0001 C CNN
 F 4 "Header for I2S Debug" H 4600 1100 50  0001 C CNN "Description"
@@
 Wire Wire Line
 	4350 1300 4400 1300
+Text Label 4350 1000 2    50   ~ 0
+I2S_CK
+Text Label 4350 1200 2    50   ~ 0
+I2S_WS
 Text Label 4350 1100 2    50   ~ 0
-I2S_CK
-Text Label 4350 1000 2    50   ~ 0
-I2S_WS
-Text Label 4350 1200 2    50   ~ 0
 I2S_SD
 Wire Wire Line
@@
 L Device:R_Small R31
 U 1 1 61277C8A
-P 3500 4950
-F 0 "R31" V 3435 4945 50  0000 C CNN
-F 1 "470" V 3570 4945 50  0000 C CNN
-F 2 "Resistor_SMD:R_0603_1608Metric" H 3500 4950 50  0001 C CNN
-F 3 "~" H 3500 4950 50  0001 C CNN
-	1    3500 4950
+P 3500 4450
+F 0 "R31" V 3435 4445 50  0000 C CNN
+F 1 "470" V 3570 4445 50  0000 C CNN
+F 2 "Resistor_SMD:R_0603_1608Metric" H 3500 4450 50  0001 C CNN
+F 3 "~" H 3500 4450 50  0001 C CNN
+	1    3500 4450
 	0    1    1    0
 $EndComp
@@
 	3600 3950 3650 3950
 Wire Wire Line
-	3650 4950 3600 4950
+	3650 4450 3600 4450
 Wire Wire Line
 	7200 5000 7250 5000
@@
 Wire Wire Line
 	10300 1150 10300 1100
-Text HLabel 3350 3350 2    50   Output ~ 0
+Text HLabel 3400 1850 2    50   Output ~ 0
 SPI_INT
-Wire Wire Line
-	3350 3350 3250 3350
 $Comp
 L Switch:SW_Push_Dual SW5
@@
 $EndComp
 $Comp
-L power:+3.3VDAC #PWR?
+L power:+3.3VDAC #PWR0103
 U 1 1 607E677E
 P 9600 4150
-F 0 "#PWR?" H 9750 4100 50  0001 C CNN
+F 0 "#PWR0103" H 9750 4100 50  0001 C CNN
 F 1 "+3.3VDAC" H 9620 4293 50  0000 C CNN
 F 2 "" H 9600 4150 50  0001 C CNN
@@
 	1    0    0    -1
 $EndComp
+NoConn ~ 3250 5650
+NoConn ~ 3250 4950
+Wire Wire Line
+	3400 1850 3250 1850
+NoConn ~ 3250 3350
 $EndSCHEMATC
