File: midi_dac.sch (KiCad schematic (older format))
At the start: 70 parts, among them CON1 SN49B12B, J10 USB_A, J11 Conn_02x05_Odd_Even, J12 Conn_01x03_Male, J13 Conn_01x04_Male, J9 Conn_01x05_Male, SW4 SW_Push_Dual, SW5 SW_Push_Dual, SW6 SW_Push_Dual, U5 STM32F407VGT6, U6 PCM5102, U7 STMPS2141STR, U9 USBLC6-2SC6, Y2 8MHz

Commit message: Huge progress on routing
Parts:
- removed D2: BLUE_LED, LED_SMD:LED_0603_1608Metric, symbol Device:LED
- removed D3: GREEN_LED, LED_SMD:LED_0603_1608Metric, symbol Device:LED
- removed D4: ORA_LED, LED_SMD:LED_0603_1608Metric, symbol Device:LED
- removed D5: RED_LED, LED_SMD:LED_0603_1608Metric, symbol Device:LED
- removed J11: Conn_02x05_Odd_Even, Connector_PinHeader_2.54mm:PinHeader_2x05_P2.54mm_Vertical, symbol Connector_Generic:Conn_02x05_Odd_Even
- removed R25, R26, R27, R28: 75, Resistor_SMD:R_0603_1608Metric, symbol Device:R_Small
- added J11: Conn_02x10_Odd_Even, Connector_PinHeader_1.27mm:PinHeader_2x10_P1.27mm_Vertical, symbol Connector_Generic:Conn_02x10_Odd_Even
Connections:
- net +3.3VA: now also J11.1 (Pin_1)
- net GND: now also J11.10 (Pin_10), J11.12 (Pin_12), J11.14 (Pin_14), J11.16 (Pin_16), J11.18 (Pin_18), J11.20 (Pin_20), J11.4 (Pin_4), J11.6 (Pin_6), J11.8 (Pin_8)
- net NRST: now also J11.15 (Pin_15)
- net SWCLK: now also J11.9 (Pin_9)
- net SWDIO: now also J11.7 (Pin_7)
- net SWO: now also J11.13 (Pin_13)
- net GPIO_OUTPUT_D12: no longer names the net of U5.59 (PD12)
- net GPIO_OUTPUT_D13: no longer names the net of U5.60 (PD13)
- net GPIO_OUTPUT_D14: no longer names the net of U5.61 (PD14)
- net GPIO_OUTPUT_D15: no longer names the net of U5.62 (PD15)
- no-connect marks 60 -> 68
