File: midi_dac.sch (KiCad schematic (older format))
At the start: 62 parts, among them CON1 SN49B12B, J10 USB_A, J11 Conn_02x10_Odd_Even, J12 Conn_01x03_Male, J13 Conn_01x04_Male, J9 Conn_01x05_Male, SW4 SW_Push_Dual, SW5 SW_Push_Dual, SW6 SW_Push_Dual, U5 STM32F407VGT6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

Commit message: Finish initial layout
Parts:
- removed J11: Conn_02x10_Odd_Even, Connector_PinHeader_1.27mm:PinHeader_2x10_P1.27mm_Vertical, symbol Connector_Generic:Conn_02x10_Odd_Even
- removed SW4, SW5, SW6: SW_Push_Dual, Button_Switch_SMD:SW_SPST_EVPBF, symbol Switch:SW_Push_Dual
- added J11: Conn_02x05_Odd_Even, Connector_PinHeader_1.27mm:PinHeader_2x05_P1.27mm_Vertical, symbol Connector_Generic:Conn_02x05_Odd_Even
- added J16, J17, J18: Conn_01x02_Male, Connector_PinHeader_2.54mm:PinHeader_1x02_P2.54mm_Vertical, symbol Connector:Conn_01x02_Male
- added R27: 300k, Resistor_SMD:R_0603_1608Metric, symbol Device:R_Small
- added R28: 200k, Resistor_SMD:R_0603_1608Metric, symbol Device:R_Small
Connections:
- net labels removed: +3.3VA
- wire segments 288 -> 293
- no-connect marks 68 -> 65

Commit message: PCB changes
Parts:
- removed J13: Conn_01x04_Male, Connector_PinHeader_2.54mm:PinHeader_1x04_P2.54mm_Vertical, symbol Connector:Conn_01x04_Male
- removed J9: Conn_01x05_Male, Connector_PinHeader_2.54mm:PinHeader_1x05_P2.54mm_Vertical, symbol Connector:Conn_01x05_Male
- added J13: Conn_01x03_Male, Connector_PinHeader_2.54mm:PinHeader_1x03_P2.54mm_Vertical, symbol Connector:Conn_01x03_Male
- added J9: Conn_01x04_Male, Connector_PinHeader_2.54mm:PinHeader_1x04_P2.54mm_Vertical, symbol Connector:Conn_01x04_Male
- added R47: 0, Resistor_SMD:R_0603_1608Metric, symbol Device:R_Small
- added R50: 47k, Resistor_SMD:R_0603_1608Metric, symbol Device:R_Small
- added R53: 97k, Resistor_SMD:R_0603_1608Metric, symbol Device:R_Small
- J10: Digi-Key_PN (none) -> 67643-3910
- U5: Digi-Key_PN (none) -> STM32F407VGT6
- U6: Digi-Key_PN (none) -> PCM5102APWR
- U9: Digi-Key_PN (none) -> USBLC6-2SC6
- Y2: Digi-Key_PN (none) -> ASDDV-8.000MHZ-LR-T
Connections:
- net +3.3VDAC: now also U6.1 (CPVDD)
- net +3V3: no longer U6.1 (CPVDD), Y2.4
- net GND: now also Y2.4, J13.1 (Pin_1), J9.1 (Pin_1), R47.1, R53.2; no longer J10.5 (Shield)
- net I2S_CK: now also J9.4 (Pin_4)
- net I2S_SD: now also J9.2 (Pin_2)
- net I2S_WS: now also J9.3 (Pin_3)
- net SOFT_MUTE: now also U5.55 (PD8); no longer U5.45 (PE14)
- net UART4_RX: now also J13.3 (Pin_3)
- net UART4_TX: now also J13.2 (Pin_2)
- net USB_DM: no longer R35.2
- net USB_DP: no longer R34.2
- net USB_FS_DM: no longer U9.6 (IO1)
- net USB_FS_DP: no longer U9.4 (IO2)
- net USB_FS_VBUS: now also R50.2, R53.1; no longer C44.1, J10.1 (VBUS), U7.1 (OUT)
- net USB_VBUS_EN: now also U5.67 (PA8); no longer U5.69 (PA10)
- new net: R34.2, U9.4 (IO2)
- new net: R35.2, U9.6 (IO1)
- new net: J10.5 (Shield), R47.2
- new net USB_POWER: C44.1, J10.1 (VBUS), R50.1, U7.1 (OUT)
- no-connect marks 65 -> 64
Other:
- moved on the sheet: R34, R35

Commit message: Updated
Parts:
- J11: footprint Connector_PinHeader_1.27mm:PinHeader_2x05_P1.27mm_Vertical -> Connector_PinHeader_1.27mm:PinHeader_2x05_P1.27mm_Vertical_SMD
Connections:
- net +5V: no longer C57.1, U9.5 (VBUS)
- net USB_POWER: now also C57.1, U9.5 (VBUS)
Changed lines of the file:
@@
-	1    0    0    -1
-$EndComp
-$Comp
-L power:+5V #PWR057
-U 1 1 606180F0
-P 5050 5050
-F 0 "#PWR057" H 5050 4900 50  0001 C CNN
-F 1 "+5V" H 5065 5223 50  0000 C CNN
-F 2 "" H 5050 5050 50  0001 C CNN
-F 3 "" H 5050 5050 50  0001 C CNN
-	1    5050 5050
 	1    0    0    -1
 $EndComp
@@
 F 4 "5.2 V" H 5550 6100 50  0001 C CNN "Min Voltage Rating"
 	1    5550 6100
-	1    0    0    -1
-$EndComp
-$Comp
-L power:+5V #PWR099
-U 1 1 6065220C
-P 5550 5950
-F 0 "#PWR099" H 5550 5800 50  0001 C CNN
-F 1 "+5V" H 5565 6123 50  0000 C CNN
-F 2 "" H 5550 5950 50  0001 C CNN
-F 3 "" H 5550 5950 50  0001 C CNN
-	1    5550 5950
 	1    0    0    -1
 $EndComp
@@
 F 0 "J11" H 5400 4567 50  0000 C CNN
 F 1 "Conn_02x05_Odd_Even" H 5700 4500 50  0000 C CNN
-F 2 "Connector_PinHeader_1.27mm:PinHeader_2x05_P1.27mm_Vertical" H 5350 4150 50  0001 C CNN
+F 2 "Connector_PinHeader_1.27mm:PinHeader_2x05_P1.27mm_Vertical_SMD" H 5350 4150 50  0001 C CNN
 F 3 "~" H 5350 4150 50  0001 C CNN
 	1    5350 4150
@@
 	-1   0    0    1
 $EndComp
+Text Label 5050 5050 0    50   ~ 0
+USB_POWER
+Text Label 5550 5950 0    50   ~ 0
+USB_POWER
 $EndSCHEMATC
