File: digidraw.sch (KiCad schematic (older format))
At the start: 44 parts, among them J1 USB_B_Micro, J2 Barrel_Jack, Q1 FDD5614P, U1 TPS63070RNMR, U2 LM117_TO3, U8 LM117_TO3

Commit message: Finish schematic
Parts:
- C1, C2, C3, C4, C5: Min Voltage Rating (none) -> 16 V
- C48, C49, C50, C51, C52, C6: Min Voltage Rating (none) -> 5.2 V
- C53, C54, C55, C56: Min Voltage Rating (none) -> 3.3 V
- D6: Description (none) -> Debug LED
- F1: Description (none) -> Input current fuse
- H1, H2, H3, H4: Description (none) -> Mounting Holes
- J1: Description (none) -> USB B micro for power
- J2: Description (none) -> Barrel jack for power (maybe)
- L1: Description (none) -> Buck/Boost converter inductor
- Q1: Description (none) -> MOSFET for bias protection
- U1: Description (none) -> Buck/boost converter
- U2, U8: Description (none) -> Converters for +5 to +3.3 V
Changed lines of the file:
@@
 F 2 "digikey-footprints:Barrel_Jack_5.5mmODx2.1mmID_PJ-202A" H 5650 1360 50  0001 C CNN
 F 3 "~" H 5650 1360 50  0001 C CNN
+F 4 "Barrel jack for power (maybe)" H 5600 1400 50  0001 C CNN "Description"
 	1    5600 1400
 	1    0    0    -1
@@
 F 2 "MountingHole:MountingHole_4.3mm_M4_Pad_Via" H 5000 5250 50  0001 C CNN
 F 3 "~" H 5000 5250 50  0001 C CNN
+F 4 "Mounting Holes" H 5000 5250 50  0001 C CNN "Description"
 	1    5000 5250
 	1    0    0    -1
@@
 F 2 "MountingHole:MountingHole_4.3mm_M4_Pad_Via" H 5000 5800 50  0001 C CNN
 F 3 "~" H 5000 5800 50  0001 C CNN
+F 4 "Mounting Holes" H 5000 5800 50  0001 C CNN "Description"
 	1    5000 5800
 	1    0    0    -1
@@
 F 2 "MountingHole:MountingHole_4.3mm_M4_Pad_Via" H 5000 6350 50  0001 C CNN
 F 3 "~" H 5000 6350 50  0001 C CNN
+F 4 "Mounting Holes" H 5000 6350 50  0001 C CNN "Description"
 	1    5000 6350
 	1    0    0    -1
@@
 F 2 "MountingHole:MountingHole_4.3mm_M4_Pad_Via" H 5000 6950 50  0001 C CNN
 F 3 "~" H 5000 6950 50  0001 C CNN
+F 4 "Mounting Holes" H 5000 6950 50  0001 C CNN "Description"
 	1    5000 6950
 	1    0    0    -1
@@
 F 2 "Connector_USB:USB_Micro-B_Molex-105017-0001" H 4200 1250 50  0001 C CNN
 F 3 "~" H 4200 1250 50  0001 C CNN
+F 4 "USB B micro for power" H 4050 1300 50  0001 C CNN "Description"
 	1    4050 1300
 	1    0    0    -1
@@
 F 2 "Fuse:Fuse_0805_2012Metric" H 1200 2950 50  0001 C CNN
 F 3 "~" H 1200 2950 50  0001 C CNN
+F 4 "Input current fuse" H 1200 2950 50  0001 C CNN "Description"
 	1    1200 2950
 	1    0    0    -1
@@
 F 2 "Capacitor_SMD:C_0805_2012Metric" H 1400 3150 50  0001 C CNN
 F 3 "~" H 1400 3150 50  0001 C CNN
+F 4 "16 V" H 1400 3150 50  0001 C CNN "Min Voltage Rating"
 	1    1400 3150
 	1    0    0    -1
@@
 F 2 "Diode_SMD:D_0603_1608Metric" V 2900 3150 50  0001 C CNN
 F 3 "~" V 2900 3150 50  0001 C CNN
+F 4 "Debug LED" H 2900 3150 50  0001 C CNN "Description"
 	1    2900 3150
 	0    1    1    0
@@
 F 2 "Capacitor_SMD:C_0805_2012Metric" H 3300 3150 50  0001 C CNN
 F 3 "~" H 3300 3150 50  0001 C CNN
+F 4 "16 V" H 3300 3150 50  0001 C CNN "Min Voltage Rating"
 	1    3300 3150
 	1    0    0    -1
@@
 F 2 "Capacitor_SMD:C_0805_2012Metric" H 3600 3150 50  0001 C CNN
 F 3 "~" H 3600 3150 50  0001 C CNN
+F 4 "16 V" H 3600 3150 50  0001 C CNN "Min Voltage Rating"
 	1    3600 3150
 	1    0    0    -1
@@
 F 30 "+125°C" H 4500 6150 50  0001 L CNN "temperature range high"
 F 31 "-40°C" H 4500 6250 50  0001 L CNN "temperature range low"
+F 32 "Buck/boost converter" H 4500 2950 50  0001 C CNN "Description"
 	1    4500 2950
 	1    0    0    -1
@@
 F 2 "Capacitor_SMD:C_0603_1608Metric" H 4000 3050 50  0001 C CNN
 F 3 "~" H 4000 3050 50  0001 C CNN
+F 4 "16 V" H 4000 3050 50  0001 C CNN "Min Voltage Rating"
 	1    4000 3050
 	1    0    0    -1
@@
 F 2 "Capacitor_SMD:C_0805_2012Metric" H 4100 3300 50  0001 C CNN
 F 3 "~" H 4100 3300 50  0001 C CNN
+F 4 "16 V" H 4100 3300 50  0001 C CNN "Min Voltage Rating"
 	1    4100 3300
 	1    0    0    -1
@@
 F 2 "Inductor_SMD:L_0603_1608Metric" H 4500 3400 50  0001 C CNN
 F 3 "~" H 4500 3400 50  0001 C CNN
+F 4 "Buck/Boost converter inductor" H 4500 3400 50  0001 C CNN "Description"
 	1    4500 3400
 	-1   0    0    1
@@
 F 2 "Capacitor_SMD:C_0603_1608Metric" H 5950 3050 50  0001 C CNN
 F 3 "~" H 5950 3050 50  0001 C CNN
+F 4 "5.2 V" H 5950 3050 50  0001 C CNN "Min Voltage Rating"
 	1    5950 3050
 	1    0    0    -1
@@
 F 2 "Capacitor_SMD:C_0805_2012Metric" H 6750 3100 50  0001 C CNN
 F 3 "~" H 6750 3100 50  0001 C CNN
+F 4 "5.2 V" H 6750 3100 50  0001 C CNN "Min Voltage Rating"
 	1    6750 3100
 	1    0    0    -1
@@
 F 2 "Capacitor_SMD:C_0805_2012Metric" H 7050 3100 50  0001 C CNN
 F 3 "~" H 7050 3100 50  0001 C CNN
+F 4 "5.2 V" H 7050 3100 50  0001 C CNN "Min Voltage Rating"
 	1    7050 3100
 	1    0    0    -1
@@
 F 2 "Capacitor_SMD:C_0805_2012Metric" H 7350 3100 50  0001 C CNN
 F 3 "~" H 7350 3100 50  0001 C CNN
+F 4 "5.2 V" H 7350 3100 50  0001 C CNN "Min Voltage Rating"
 	1    7350 3100
 	1    0    0    -1
@@
 F 2 "Package_TO_SOT_THT:TO-3" H 8400 3750 50  0001 C CIN
 F 3 "http://www.ti.com/lit/ds/symlink/lm317.pdf" H 8400 3550 50  0001 C CNN
+F 4 "Converters for +5 to +3.3 V" H 8400 3550 50  0001 C CNN "Description"
 	1    8400 3550
 	1    0    0    -1
@@
 F 2 "Capacitor_SMD:C_0805_2012Metric" H 7800 4900 50  0001 C CNN
 F 3 "~" H 7800 4900 50  0001 C CNN
+F 4 "5.2 V" H 7800 4900 50  0001 C CNN "Min Voltage Rating"
 	1    7800 4900
 	1    0    0    -1
@@
 F 2 "Capacitor_SMD:C_0805_2012Metric" H 8850 5000 50  0001 C CNN
 F 3 "~" H 8850 5000 50  0001 C CNN
+F 4 "3.3 V" H 8850 5000 50  0001 C CNN "Min Voltage Rating"
 	1    8850 5000
 	1    0    0    -1
@@
 F 2 "Capacitor_SMD:C_0603_1608Metric" H 9200 5000 50  0001 C CNN
 F 3 "~" H 9200 5000 50  0001 C CNN
+F 4 "3.3 V" H 9200 5000 50  0001 C CNN "Min Voltage Rating"
 	1    9200 5000
 	1    0    0    -1
@@
 F 2 "Capacitor_SMD:C_0805_2012Metric" H 8000 3700 50  0001 C CNN
 F 3 "~" H 8000 3700 50  0001 C CNN
+F 4 "5.2 V" H 8000 3700 50  0001 C CNN "Min Voltage Rating"
 	1    8000 3700
 	1    0    0    -1
@@
 F 2 "Capacitor_SMD:C_0805_2012Metric" H 9150 3750 50  0001 C CNN
 F 3 "~" H 9150 3750 50  0001 C CNN
+F 4 "3.3 V" H 9150 3750 50  0001 C CNN "Min Voltage Rating"
 	1    9150 3750
 	1    0    0    -1
@@
 F 2 "Capacitor_SMD:C_0603_1608Metric" H 9500 3750 50  0001 C CNN
 F 3 "~" H 9500 3750 50  0001 C CNN
+F 4 "3.3 V" H 9500 3750 50  0001 C CNN "Min Voltage Rating"
 	1    9500 3750
 	1    0    0    -1
@@
 F 32 "19ns" H 2400 6850 50  0001 L CNN "turn off delay time"
 F 33 "7ns" H 2400 6950 50  0001 L CNN "turn on delay time"
+F 34 "MOSFET for bias protection" H 2400 3350 50  0001 C CNN "Description"
 	1    2400 3350
 	0    -1   -1   0
@@
 F 2 "Package_TO_SOT_THT:TO-3" H 8200 4950 50  0001 C CIN
 F 3 "http://www.ti.com/lit/ds/symlink/lm317.pdf" H 8200 4750 50  0001 C CNN
+F 4 "Converters for +5 to +3.3 V" H 8200 4750 50  0001 C CNN "Description"
 	1    8200 4750
 	1    0    0    -1

Commit message: Get everything on board, use buck converter, chnage lm317 footprint
Parts:
- removed R47: 542, Resistor_SMD:R_0603_1608Metric, symbol Device:R_Small
- removed R50: 330, Resistor_SMD:R_0603_1608Metric, symbol Device:R_Small
- removed U2, U8: LM117_TO3, Package_TO_SOT_THT:TO-3, symbol Regulator_Linear:LM117_TO3
- added L2: L_Small, Inductor_SMD:L_0603_1608Metric, symbol Device:L_Small
- added U2: V7803-1500R, v7803:CONV_V7803-1500R, symbol V7803-1500R:V7803-1500R
- added U8: LM317KCS, lm317_ti:LM317KCS, symbol lm317_ti:LM317KCS
- C51: footprint Capacitor_SMD:C_0805_2012Metric -> Capacitor_SMD:C_0603_1608Metric; Min Voltage Rating 5.2 V -> (none)
- C53: value 100n -> 10u; footprint Capacitor_SMD:C_0805_2012Metric -> Capacitor_SMD:C_0603_1608Metric; Min Voltage Rating 3.3 V -> (none)
- C55: value 10u -> 22u; Min Voltage Rating 3.3 V -> (none)
Connections:
- wire segments 160 -> 161
Other:
- moved on the sheet: C54, C56, R48, R51

Commit message: Huge progress on routing
Parts:
- added D2, D3: LED, LED_SMD:LED_0603_1608Metric, symbol Device:LED
- added R25: 208, Resistor_SMD:R_0603_1608Metric, symbol Device:R_Small
- added R26: 100, Resistor_SMD:R_0603_1608Metric, symbol Device:R_Small
Connections:
- net +3V3: now also D3.2 (A)
- net +5V: now also D2.2 (A)
- net GND: now also R25.2, R26.2
- new net: D2.1 (K), R25.1
- new net: D3.1 (K), R26.1
Changed lines of the file:
@@
 Connection ~ 9900 3550
 Connection ~ 9550 3550
+$Comp
+L Device:LED D2
+U 1 1 6061A107
+P 8950 1700
+F 0 "D2" V 8989 1583 50  0000 R CNN
+F 1 "LED" V 8898 1583 50  0000 R CNN
+F 2 "LED_SMD:LED_0603_1608Metric" H 8950 1700 50  0001 C CNN
+F 3 "~" H 8950 1700 50  0001 C CNN
+	1    8950 1700
+	0    -1   -1   0
+$EndComp
+$Comp
+L Device:LED D3
+U 1 1 6061A674
+P 9250 1700
+F 0 "D3" V 9289 1583 50  0000 R CNN
+F 1 "LED" V 9198 1583 50  0000 R CNN
+F 2 "LED_SMD:LED_0603_1608Metric" H 9250 1700 50  0001 C CNN
+F 3 "~" H 9250 1700 50  0001 C CNN
+	1    9250 1700
+	0    -1   -1   0
+$EndComp
+$Comp
+L power:+3.3V #PWR092
+U 1 1 6061BC34
+P 9250 1550
+F 0 "#PWR092" H 9250 1400 50  0001 C CNN
+F 1 "+3.3V" H 9265 1723 50  0000 C CNN
+F 2 "" H 9250 1550 50  0001 C CNN
+F 3 "" H 9250 1550 50  0001 C CNN
+	1    9250 1550
+	1    0    0    -1
+$EndComp
+$Comp
+L power:+5V #PWR018
+U 1 1 6061CBC5
+P 8950 1550
+F 0 "#PWR018" H 8950 1400 50  0001 C CNN
+F 1 "+5V" H 8965 1723 50  0000 C CNN
+F 2 "" H 8950 1550 50  0001 C CNN
+F 3 "" H 8950 1550 50  0001 C CNN
+	1    8950 1550
+	1    0    0    -1
+$EndComp
+$Comp
+L Device:R_Small R25
+U 1 1 6061DEFB
+P 8950 2000
+F 0 "R25" H 9009 2046 50  0000 L CNN
+F 1 "208" H 9009 1955 50  0000 L CNN
+F 2 "Resistor_SMD:R_0603_1608Metric" H 8950 2000 50  0001 C CNN
+F 3 "~" H 8950 2000 50  0001 C CNN
+	1    8950 2000
+	1    0    0    -1
+$EndComp
+Wire Wire Line
+	8950 1900 8950 1850
+$Comp
+L Device:R_Small R26
+U 1 1 60623EDE
+P 9250 2000
+F 0 "R26" H 9309 2046 50  0000 L CNN
+F 1 "100" H 9309 1955 50  0000 L CNN
+F 2 "Resistor_SMD:R_0603_1608Metric" H 9250 2000 50  0001 C CNN
+F 3 "~" H 9250 2000 50  0001 C CNN
+	1    9250 2000
+	1    0    0    -1
+$EndComp
+Wire Wire Line
+	9250 1900 9250 1850
+$Comp
+L power:GND #PWR083
+U 1 1 6062AFBA
+P 8950 2150
+F 0 "#PWR083" H 8950 1900 50  0001 C CNN
+F 1 "GND" H 8955 1977 50  0000 C CNN
+F 2 "" H 8950 2150 50  0001 C CNN
+F 3 "" H 8950 2150 50  0001 C CNN
+	1    8950 2150
+	1    0    0    -1
+$EndComp
+Wire Wire Line
+	8950 2150 8950 2100
+$Comp
+L power:GND #PWR0104
+U 1 1 60631A63
+P 9250 2150
+F 0 "#PWR0104" H 9250 1900 50  0001 C CNN
+F 1 "GND" H 9255 1977 50  0000 C CNN
+F 2 "" H 9250 2150 50  0001 C CNN
+F 3 "" H 9250 2150 50  0001 C CNN
+	1    9250 2150
+	1    0    0    -1
+$EndComp
+Wire Wire Line
+	9250 2150 9250 2100
 $EndSCHEMATC

Commit message: Documentation for submission
Parts:
- C55: Min Voltage Rating (none) -> 3.3 V
Changed lines of the file:
@@
 F 2 "Capacitor_SMD:C_0603_1608Metric" H 9700 5150 50  0001 C CNN
 F 3 "~" H 9700 5150 50  0001 C CNN
+F 4 "3.3 V" H 9700 5150 50  0001 C CNN "Min Voltage Rating"
 	1    9700 5150
 	1    0    0    -1

Commit message: PCB changes
Parts:
- removed F1: 3, Fuse:Fuse_0805_2012Metric, symbol Device:Fuse_Small
- D2, D3: Digi-Key_PN (none) -> AA1608SURSK
- D6: Digi-Key_PN (none) -> CDBU0320
- J1: Digi-Key_PN (none) -> 105017-0001
- J2: Digi-Key_PN (none) -> PJ-202A
- L1: footprint Inductor_SMD:L_0603_1608Metric -> custom_fp:InductorWEPD; Digi-Key_PN (none) -> 7447707015
- L2: value L_Small -> 10u; Digi-Key_PN (none) -> MLZ1608E100MT
- Q1: Digi-Key_PN (none) -> FDD5614P
- U1: Digi-Key_PN (none) -> TPS63070RNMR
- U2: Digi-Key_PN (none) -> V7803-1500R
- U8: Digi-Key_PN (none) -> LM317KCS
Connections:
- net VIN: now also C1.1, D1.1, Q1.4 (D)
Changed lines of the file:
@@
 F 3 "~" H 5650 1360 50  0001 C CNN
 F 4 "Barrel jack for power (maybe)" H 5600 1400 50  0001 C CNN "Description"
+F 5 "PJ-202A" H 5600 1400 50  0001 C CNN "Digi-Key_PN"
 	1    5600 1400
 	1    0    0    -1
@@
 F 3 "~" H 4200 1250 50  0001 C CNN
 F 4 "USB B micro for power" H 4050 1300 50  0001 C CNN "Description"
+F 5 "105017-0001" H 4050 1300 50  0001 C CNN "Digi-Key_PN"
 	1    4050 1300
 	1    0    0    -1
@@
 Wire Wire Line
 	3050 5950 2250 5950
-$Comp
-L Device:Fuse_Small F1
-U 1 1 60805B60
-P 1200 2950
-F 0 "F1" H 1200 3135 50  0000 C CNN
-F 1 "3" H 1200 3044 50  0000 C CNN
-F 2 "Fuse:Fuse_0805_2012Metric" H 1200 2950 50  0001 C CNN
-F 3 "~" H 1200 2950 50  0001 C CNN
-F 4 "Input current fuse" H 1200 2950 50  0001 C CNN "Description"
-	1    1200 2950
-	1    0    0    -1
-$EndComp
 Text Label 950  2950 1    50   ~ 0
 VIN
-Wire Wire Line
-	950  2950 1100 2950
 $Comp
 L Device:C_Small C1
@@
 Wire Wire Line
 	1400 3050 1400 2950
-Wire Wire Line
-	1400 2950 1300 2950
 $Comp
 L power:GND #PWR01
@@
 F 3 "~" V 2900 3150 50  0001 C CNN
 F 4 "Debug LED" H 2900 3150 50  0001 C CNN "Description"
+F 5 "CDBU0320" H 2900 3150 50  0001 C CNN "Digi-Key_PN"
 	1    2900 3150
 	0    1    1    0
@@
 F 31 "-40°C" H 4500 6250 50  0001 L CNN "temperature range low"
 F 32 "Buck/boost converter" H 4500 2950 50  0001 C CNN "Description"
+F 33 "TPS63070RNMR" H 4500 2950 50  0001 C CNN "Digi-Key_PN"
 	1    4500 2950
 	1    0    0    -1
@@
 F 0 "L1" H 4600 3350 50  0000 R CNN
 F 1 "1.5u" H 4700 3450 50  0000 R CNN
-F 2 "Inductor_SMD:L_0603_1608Metric" H 4500 3400 50  0001 C CNN
+F 2 "custom_fp:InductorWEPD" H 4500 3400 50  0001 C CNN
 F 3 "~" H 4500 3400 50  0001 C CNN
 F 4 "Buck/Boost converter inductor" H 4500 3400 50  0001 C CNN "Description"
+F 5 "7447707015" H 4500 3400 50  0001 C CNN "Digi-Key_PN"
 	1    4500 3400
 	-1   0    0    1
@@
 F 33 "7ns" H 2400 6950 50  0001 L CNN "turn on delay time"
 F 34 "MOSFET for bias protection" H 2400 3350 50  0001 C CNN "Description"
+F 35 "FDD5614P" H 2400 3350 50  0001 C CNN "Digi-Key_PN"
 	1    2400 3350
 	0    -1   -1   0
@@
 F 5 "1.03" H 8500 5050 50  0001 L BNN "PARTREV"
 F 6 "MANUFACTURER RECOMMENDATIONS" H 8500 5050 50  0001 L BNN "STANDARD"
+F 7 "V7803-1500R" H 8500 5050 50  0001 C CNN "Digi-Key_PN"
 	1    8500 5050
 	1    0    0    -1
@@
 P 9550 4950
 F 0 "L2" V 9369 4950 50  0000 C CNN
-F 1 "L_Small" V 9460 4950 50  0000 C CNN
+F 1 "10u" V 9460 4950 50  0000 C CNN
 F 2 "Inductor_SMD:L_0603_1608Metric" H 9550 4950 50  0001 C CNN
 F 3 "~" H 9550 4950 50  0001 C CNN
+F 4 "MLZ1608E100MT" H 9550 4950 50  0001 C CNN "Digi-Key_PN"
 	1    9550 4950
 	0    1    1    0
@@
 F 2 "lm317_ti:LM317KCS" H 8600 3590 60  0001 C CNN
 F 3 "" H 8600 3650 60  0000 C CNN
+F 4 "LM317KCS" H 8600 3650 50  0001 C CNN "Digi-Key_PN"
 	1    8600 3650
 	1    0    0    -1
@@
 F 2 "LED_SMD:LED_0603_1608Metric" H 8950 1700 50  0001 C CNN
 F 3 "~" H 8950 1700 50  0001 C CNN
+F 4 "AA1608SURSK" H 8950 1700 50  0001 C CNN "Digi-Key_PN"
 	1    8950 1700
 	0    -1   -1   0
@@
 F 2 "LED_SMD:LED_0603_1608Metric" H 9250 1700 50  0001 C CNN
 F 3 "~" H 9250 1700 50  0001 C CNN
+F 4 "AA1608SURSK" H 9250 1700 50  0001 C CNN "Digi-Key_PN"
 	1    9250 1700
 	0    -1   -1   0
@@
 Wire Wire Line
 	9250 2150 9250 2100
+Wire Wire Line
+	950  2950 1400 2950
 $EndSCHEMATC
