File: digidraw.kicad_pcb (KiCad board)
At the start: 2 copper layers, 140 x 100 mm, 152 parts, among them CON1 SN49B12B, J1 USB_B_Micro, J10 USB_A, J11 Conn_02x05_Odd_Even, J12 Conn_01x03_Male, J13 Conn_01x03_Male, J14 Conn_01x02_Male, J15 Conn_01x02_Male, J16 Conn_01x02_Male, J17 Conn_01x02_Male, J18 Conn_01x02_Male, J19 Conn_01x02_Male, J2 Barrel_Jack, J3 Conn_02x05_Odd_Even, J4 Conn_01x06_Male, J5 Conn_01x05_Male, J6 Conn_01x04_Male, J7 Conn_01x09_Male, J8 Conn_01x04_Male, J9 Conn_01x04_Male, Q1 FDD5614P, U1 TPS63070RNMR, U2 V7803-1500R, U3 STM32F051R8T6, U4 CAT24C256, U5 STM32F407VGT6, U6 PCM5102, U7 STMPS2141STR, U8 LM317KCS, U9 USBLC6-2SC6, Y1 8MHz, Y2 8MHz

Commit message: Update pcb layout
Parts:
- moved C4 3.64 mm to (178.4, 89.3), turned to 270 degrees
- moved C6 1.00 mm to (178.4, 92.7), turned to 90 degrees
Routing:
- net Net-(C2-Pad1): track 25.9 -> 27.8 mm
- net Net-(C48-Pad1): track 104.2 -> 105.1 mm
- net GND: track 236.6 -> 237.0 mm, vias 110 -> 109
- net Net-(L1-Pad2): vias 0 -> 2
- net Net-(L1-Pad1): vias 0 -> 2

Commit message: Updated
Parts:
- J11, J3: footprint Connector_PinHeader_1.27mm:PinHeader_2x05_P1.27mm_Vertical -> Connector_PinHeader_1.27mm:PinHeader_2x05_P1.27mm_Vertical_SMD
- moved C57 11.6 mm to (95.7, 77.1), turned to 0 degrees
- moved J3 3.22 mm to (86.8, 151.6)
- moved J11 2.98 mm to (66.3, 99.9)
- moved C28 0.81 mm to (80.5, 114.9)
- moved C30 0.81 mm to (84.6, 114.2)
- moved Y2 0.81 mm to (82.7, 111.8)
- moved R42 0.81 mm to (85.4, 111.9)
Connections:
- C57 pad 1: +5V -> /midi_dac/USB_POWER
- U9 pad 5: +5V -> /midi_dac/USB_POWER
Routing:
- net +5V: track 133.0 -> 96.6 mm
- net /midi_dac/NRST: track 42.7 -> 53.2 mm
- net /midi_dac/USB_POWER: track 25.4 -> 34.4 mm
- net GND: track 237.0 -> 245.7 mm, vias 109 -> 112
- net /user_io/NRST: track 85.6 -> 81.1 mm
- net /user_io/SWDIO: track 12.7 -> 8.79 mm
- net /user_io/SWCLK: track 13.1 -> 9.19 mm
- net /midi_dac/SWDIO: track 18.0 -> 14.8 mm
- net /midi_dac/SWCLK: track 12.8 -> 9.58 mm
- net /midi_dac/SWO: track 11.5 -> 8.74 mm
- net /midi_dac/HSE_IN: track 6.11 -> 7.10 mm
- net +3V3: track 607.5 -> 608.4 mm
