File: user_io.sch (KiCad schematic (older format))
At the start: 39 parts, among them J3 Conn_02x05_Odd_Even, J4 Conn_01x06_Male, J5 Conn_01x05_Male, J6 Conn_01x04_Male, J7 Conn_01x15_Female, J8 Conn_01x04_Male, SW1 SW_Push_Dual, SW2 SW_Push_Dual, SW3 SW_Push_Dual, U3 STM32F051R8T6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

Commit message: Work on pcb layout
Parts:
- J3: footprint Connector_PinHeader_2.54mm:PinHeader_1x38_P2.54mm_Vertical -> Connector_PinHeader_2.54mm:PinHeader_2x05_P2.54mm_Vertical
- J4: footprint Connector_PinHeader_2.54mm:PinHeader_1x38_P2.54mm_Vertical -> Connector_PinHeader_2.54mm:PinHeader_1x06_P2.54mm_Vertical
- J5: footprint Connector_PinHeader_2.54mm:PinHeader_1x38_P2.54mm_Vertical -> Connector_PinHeader_2.54mm:PinHeader_1x05_P2.54mm_Vertical
- J6: footprint Connector_PinHeader_2.54mm:PinHeader_1x38_P2.54mm_Vertical -> Connector_PinHeader_2.54mm:PinHeader_1x04_P2.54mm_Vertical
- J7: footprint Connector_PinSocket_2.54mm:PinSocket_1x07_P2.54mm_Vertical -> Connector_PinSocket_2.54mm:PinSocket_1x15_P2.54mm_Vertical
- J8: footprint Connector_PinHeader_2.54mm:PinHeader_1x08_P2.54mm_Vertical -> Connector_PinSocket_2.54mm:PinSocket_1x04_P2.54mm_Vertical
Changed lines of the file:
@@
 F 0 "J7" H 10050 2400 50  0000 C CNN
 F 1 "Conn_01x15_Female" H 10100 4050 50  0000 C CNN
-F 2 "Connector_PinSocket_2.54mm:PinSocket_1x07_P2.54mm_Vertical" H 10100 3200 50  0001 C CNN
+F 2 "Connector_PinSocket_2.54mm:PinSocket_1x15_P2.54mm_Vertical" H 10100 3200 50  0001 C CNN
 F 3 "~" H 10100 3200 50  0001 C CNN
 F 4 "Header for RA8875 pins" H 10100 3200 50  0001 C CNN "Description"
@@
 F 0 "J3" H 6850 1500 50  0000 C CNN
 F 1 "Conn_02x05_Odd_Even" H 7000 900 50  0000 C CNN
-F 2 "Connector_PinHeader_2.54mm:PinHeader_1x38_P2.54mm_Vertical" H 6800 1200 50  0001 C CNN
+F 2 "Connector_PinHeader_2.54mm:PinHeader_2x05_P2.54mm_Vertical" H 6800 1200 50  0001 C CNN
 F 3 "~" H 6800 1200 50  0001 C CNN
 F 4 "STLink header for programming/debugging" H 6800 1200 50  0001 C CNN "Description"
@@
 F 0 "J8" H 10200 4600 50  0000 R CNN
 F 1 "Conn_01x04_Male" V 10050 5150 50  0000 R CNN
-F 2 "Connector_PinHeader_2.54mm:PinHeader_1x08_P2.54mm_Vertical" H 10150 4850 50  0001 C CNN
+F 2 "Connector_PinSocket_2.54mm:PinSocket_1x04_P2.54mm_Vertical" H 10150 4850 50  0001 C CNN
 F 3 "~" H 10150 4850 50  0001 C CNN
 F 4 "Header for F0 UART Debug" H 10150 4850 50  0001 C CNN "Description"
@@
 F 0 "J6" H 9050 4600 50  0000 R CNN
 F 1 "Conn_01x04_Male" H 9200 5000 50  0000 R CNN
-F 2 "Connector_PinHeader_2.54mm:PinHeader_1x38_P2.54mm_Vertical" H 9000 4850 50  0001 C CNN
+F 2 "Connector_PinHeader_2.54mm:PinHeader_1x04_P2.54mm_Vertical" H 9000 4850 50  0001 C CNN
 F 3 "~" H 9000 4850 50  0001 C CNN
 F 4 "Header for EEPROM I2C Debug" H 9000 4850 50  0001 C CNN "Description"
@@
 F 0 "J5" H 8100 4500 50  0000 R CNN
 F 1 "Conn_01x05_Male" H 8200 5000 50  0000 R CNN
-F 2 "Connector_PinHeader_2.54mm:PinHeader_1x38_P2.54mm_Vertical" H 8050 4750 50  0001 C CNN
+F 2 "Connector_PinHeader_2.54mm:PinHeader_1x05_P2.54mm_Vertical" H 8050 4750 50  0001 C CNN
 F 3 "~" H 8050 4750 50  0001 C CNN
 F 4 "Header for subsystem SPI Debug" H 8050 4750 50  0001 C CNN "Description"
@@
 F 0 "J4" H 7350 4400 50  0000 R CNN
 F 1 "Conn_01x06_Male" H 7550 5000 50  0000 R CNN
-F 2 "Connector_PinHeader_2.54mm:PinHeader_1x38_P2.54mm_Vertical" H 7300 4750 50  0001 C CNN
+F 2 "Connector_PinHeader_2.54mm:PinHeader_1x06_P2.54mm_Vertical" H 7300 4750 50  0001 C CNN
 F 3 "~" H 7300 4750 50  0001 C CNN
 F 4 "Header for Screen SPI Debug" H 7300 4750 50  0001 C CNN "Description"

Commit message: Replace components
Parts:
- removed J7: Conn_01x15_Female, Connector_PinSocket_2.54mm:PinSocket_1x15_P2.54mm_Vertical, symbol Connector:Conn_01x15_Female
- added J7: Conn_01x09_Male, Connector_PinHeader_2.54mm:PinHeader_1x09_P2.54mm_Vertical, symbol Connector:Conn_01x09_Male
- J8: footprint Connector_PinSocket_2.54mm:PinSocket_1x04_P2.54mm_Vertical -> Connector_PinHeader_2.54mm:PinHeader_1x04_P2.54mm_Vertical
Connections:
- no-connect marks 44 -> 38
Changed lines of the file:
@@
-$EndComp
-$Comp
-L Connector:Conn_01x15_Female J7
-U 1 1 604677A6
-P 10100 3200
-F 0 "J7" H 10050 2400 50  0000 C CNN
-F 1 "Conn_01x15_Female" H 10100 4050 50  0000 C CNN
-F 2 "Connector_PinSocket_2.54mm:PinSocket_1x15_P2.54mm_Vertical" H 10100 3200 50  0001 C CNN
-F 3 "~" H 10100 3200 50  0001 C CNN
-F 4 "Header for RA8875 pins" H 10100 3200 50  0001 C CNN "Description"
-	1    10100 3200
-	1    0    0    -1
 $EndComp
 $Comp
@@
 Text Notes 6650 2150 0    50   ~ 0
 User IO to DAC SPI
-Text Label 9900 2900 2    50   ~ 0
+Text Label 10050 2800 2    50   ~ 0
 RA8875_SCK
-Text Label 9900 3000 2    50   ~ 0
+Text Label 10050 2900 2    50   ~ 0
 RA8875_MISO
-Text Label 9900 3100 2    50   ~ 0
+Text Label 10050 3000 2    50   ~ 0
 RA8875_MOSI
-Text Label 9900 3200 2    50   ~ 0
+Text Label 10050 3100 2    50   ~ 0
 RA8875_NSS
-Text Label 9900 3300 2    50   ~ 0
+Text Label 10050 3200 2    50   ~ 0
 RA8875_NRST
-Text Label 9900 3400 2    50   ~ 0
+Text Label 10050 3300 2    50   ~ 0
 RA8875_WAIT
-Text Label 9900 3500 2    50   ~ 0
+Text Label 10050 3400 2    50   ~ 0
 RA8875_INT
 Wire Wire Line
@@
 F 0 "J8" H 10200 4600 50  0000 R CNN
 F 1 "Conn_01x04_Male" V 10050 5150 50  0000 R CNN
-F 2 "Connector_PinSocket_2.54mm:PinSocket_1x04_P2.54mm_Vertical" H 10150 4850 50  0001 C CNN
+F 2 "Connector_PinHeader_2.54mm:PinHeader_1x04_P2.54mm_Vertical" H 10150 4850 50  0001 C CNN
 F 3 "~" H 10150 4850 50  0001 C CNN
 F 4 "Header for F0 UART Debug" H 10150 4850 50  0001 C CNN "Description"
@@
 RA8875_WAIT
 $Comp
-L power:+3.3V #PWR050
-U 1 1 6077D51D
-P 9350 2400
-F 0 "#PWR050" H 9350 2250 50  0001 C CNN
-F 1 "+3.3V" H 9365 2573 50  0000 C CNN
-F 2 "" H 9350 2400 50  0001 C CNN
-F 3 "" H 9350 2400 50  0001 C CNN
-	1    9350 2400
-	1    0    0    -1
-$EndComp
-$Comp
 L power:GND #PWR051
 U 1 1 6077DDED
-P 9350 2650
-F 0 "#PWR051" H 9350 2400 50  0001 C CNN
-F 1 "GND" H 9355 2477 50  0000 C CNN
-F 2 "" H 9350 2650 50  0001 C CNN
-F 3 "" H 9350 2650 50  0001 C CNN
-	1    9350 2650
-	1    0    0    -1
-$EndComp
-Wire Wire Line
-	9350 2400 9350 2500
-Wire Wire Line
-	9350 2650 9350 2600
-NoConn ~ 9900 3600
-NoConn ~ 9900 3700
-NoConn ~ 9900 3800
-NoConn ~ 9900 3900
-NoConn ~ 9900 2700
-NoConn ~ 9900 2800
-Wire Wire Line
-	9350 2600 9900 2600
-Wire Wire Line
-	9900 2500 9350 2500
+P 9450 2750
+F 0 "#PWR051" H 9450 2500 50  0001 C CNN
+F 1 "GND" H 9455 2577 50  0000 C CNN
+F 2 "" H 9450 2750 50  0001 C CNN
+F 3 "" H 9450 2750 50  0001 C CNN
+	1    9450 2750
+	1    0    0    -1
+$EndComp
 Text Label 8750 2700 0    50   ~ 0
 RA8875_NSS
@@
 Text Notes 6550 3250 0    50   ~ 0
 External Oscillator
-Text Label 7050 4550 2    50   ~ 0
+Text Label 7050 4850 2    50   ~ 0
 RA8875_NSS
 Text Label 7050 4750 2    50   ~ 0
 RA8875_MOSI
-Text Label 7050 4850 2    50   ~ 0
+Text Label 7050 4650 2    50   ~ 0
 RA8875_MISO
-Text Label 7050 4650 2    50   ~ 0
+Text Label 7050 4550 2    50   ~ 0
 RA8875_SCK
 Wire Wire Line
@@
 	1    0    0    -1
 $EndComp
+$Comp
+L Connector:Conn_01x09_Male J7
+U 1 1 60803787
+P 10250 3000
+F 0 "J7" H 10222 2932 50  0000 R CNN
+F 1 "Conn_01x09_Male" H 10650 2500 50  0000 R CNN
+F 2 "Connector_PinHeader_2.54mm:PinHeader_1x09_P2.54mm_Vertical" H 10250 3000 50  0001 C CNN
+F 3 "~" H 10250 3000 50  0001 C CNN
+	1    10250 3000
+	-1   0    0    -1
+$EndComp
+Wire Wire Line
+	9450 2500 9450 2600
+$Comp
+L power:+3.3V #PWR050
+U 1 1 6077D51D
+P 9450 2500
+F 0 "#PWR050" H 9450 2350 50  0001 C CNN
+F 1 "+3.3V" H 9465 2673 50  0000 C CNN
+F 2 "" H 9450 2500 50  0001 C CNN
+F 3 "" H 9450 2500 50  0001 C CNN
+	1    9450 2500
+	1    0    0    -1
+$EndComp
+Wire Wire Line
+	9450 2700 9450 2750
+Wire Wire Line
+	9450 2700 10050 2700
+Wire Wire Line
+	9450 2600 10050 2600
 $EndSCHEMATC

Commit message: Huge progress on routing
Parts:
- removed J3: Conn_02x05_Odd_Even, Connector_PinHeader_2.54mm:PinHeader_2x05_P2.54mm_Vertical, symbol Connector_Generic:Conn_02x05_Odd_Even
- added J3: Conn_02x10_Odd_Even, Connector_PinHeader_1.27mm:PinHeader_2x10_P1.27mm_Vertical, symbol Connector_Generic:Conn_02x10_Odd_Even
Connections:
- net +3V3: now also J3.1 (Pin_1)
- net GND: now also J3.10 (Pin_10), J3.12 (Pin_12), J3.14 (Pin_14), J3.16 (Pin_16), J3.18 (Pin_18), J3.2 (Pin_2), J3.20 (Pin_20), J3.4 (Pin_4), J3.6 (Pin_6), J3.8 (Pin_8)
- net NRST: now also J3.15 (Pin_15)
- net SWCLK: now also J3.9 (Pin_9)
- net SWDIO: now also J3.7 (Pin_7)
- no-connect marks 38 -> 41
Changed lines of the file:
@@
 	2800 2600 2650 2600
-$Comp
-L Connector_Generic:Conn_02x05_Odd_Even J3
-U 1 1 61020F75
-P 6800 1200
-F 0 "J3" H 6850 1500 50  0000 C CNN
-F 1 "Conn_02x05_Odd_Even" H 7000 900 50  0000 C CNN
-F 2 "Connector_PinHeader_2.54mm:PinHeader_2x05_P2.54mm_Vertical" H 6800 1200 50  0001 C CNN
-F 3 "~" H 6800 1200 50  0001 C CNN
-F 4 "STLink header for programming/debugging" H 6800 1200 50  0001 C CNN "Description"
-	1    6800 1200
-	1    0    0    -1
-$EndComp
 $Comp
 L power:GND #PWR028
 U 1 1 6102234A
-P 6500 1450
-F 0 "#PWR028" H 6500 1200 50  0001 C CNN
-F 1 "GND" H 6505 1277 50  0000 C CNN
-F 2 "" H 6500 1450 50  0001 C CNN
-F 3 "" H 6500 1450 50  0001 C CNN
-	1    6500 1450
-	1    0    0    -1
-$EndComp
-Wire Wire Line
-	6500 1450 6500 1400
-Wire Wire Line
-	6500 1400 6600 1400
-Wire Wire Line
-	6500 1400 6500 1200
-Wire Wire Line
-	6500 1200 6600 1200
-Connection ~ 6500 1400
-Wire Wire Line
-	6500 1200 6500 1100
-Wire Wire Line
-	6500 1100 6600 1100
-Connection ~ 6500 1200
+P 7250 1950
+F 0 "#PWR028" H 7250 1700 50  0001 C CNN
+F 1 "GND" H 7100 1900 50  0000 C CNN
+F 2 "" H 7250 1950 50  0001 C CNN
+F 3 "" H 7250 1950 50  0001 C CNN
+	1    7250 1950
+	1    0    0    -1
+$EndComp
 $Comp
 L power:+3.3V #PWR027
 U 1 1 61024D4E
-P 6500 950
-F 0 "#PWR027" H 6500 800 50  0001 C CNN
-F 1 "+3.3V" H 6515 1123 50  0000 C CNN
-F 2 "" H 6500 950 50  0001 C CNN
-F 3 "" H 6500 950 50  0001 C CNN
-	1    6500 950
-	1    0    0    -1
-$EndComp
-Wire Wire Line
-	6500 950  6500 1000
-Wire Wire Line
-	6500 1000 6600 1000
-NoConn ~ 6600 1300
-NoConn ~ 7100 1300
-NoConn ~ 7100 1200
+P 6650 950
+F 0 "#PWR027" H 6650 800 50  0001 C CNN
+F 1 "+3.3V" H 6665 1123 50  0000 C CNN
+F 2 "" H 6650 950 50  0001 C CNN
+F 3 "" H 6650 950 50  0001 C CNN
+	1    6650 950
+	1    0    0    -1
+$EndComp
 Text Label 1300 2600 2    50   ~ 0
 NRST
 Wire Wire Line
 	1300 2600 1450 2600
-Text Label 7200 1400 0    50   ~ 0
+Text Label 6700 1700 2    50   ~ 0
 NRST
-Wire Wire Line
-	7200 1400 7100 1400
-Text Label 7200 1000 0    50   ~ 0
+Text Label 6700 1300 2    50   ~ 0
 SWDIO
-Text Label 7200 1100 0    50   ~ 0
+Text Label 6700 1400 2    50   ~ 0
 SWCLK
-Wire Wire Line
-	7200 1100 7100 1100
-Wire Wire Line
-	7100 1000 7200 1000
 $Comp
 L Device:C_Small C10
@@
 Text Notes 5400 2150 0    50   ~ 0
 Reset/Boot Circuitry
-Wire Notes Line
-	6400 1650 7450 1650
 Wire Notes Line
 	7450 1650 7450 700
@@
 Wire Wire Line
 	9450 2600 10050 2600
+$Comp
+L Connector_Generic:Conn_02x10_Odd_Even J3
+U 1 1 606691DA
+P 6900 1400
+F 0 "J3" H 6950 2017 50  0000 C CNN
+F 1 "Conn_02x10_Odd_Even" V 7300 1350 50  0000 C CNN
+F 2 "Connector_PinHeader_1.27mm:PinHeader_2x10_P1.27mm_Vertical" H 6900 1400 50  0001 C CNN
+F 3 "~" H 6900 1400 50  0001 C CNN
+	1    6900 1400
+	1    0    0    -1
+$EndComp
+NoConn ~ 6700 1500
+NoConn ~ 6700 1600
+NoConn ~ 6700 1800
+NoConn ~ 6700 1900
+NoConn ~ 6700 1100
+NoConn ~ 6700 1200
+Wire Wire Line
+	6650 950  6650 1000
+Wire Wire Line
+	6650 1000 6700 1000
+Wire Wire Line
+	7250 1950 7250 1900
+Wire Wire Line
+	7250 1900 7200 1900
+Wire Wire Line
+	7200 1900 7200 1800
+Connection ~ 7200 1900
+Connection ~ 7200 1100
+Wire Wire Line
+	7200 1100 7200 1000
+Connection ~ 7200 1200
+Wire Wire Line
+	7200 1200 7200 1100
+Connection ~ 7200 1300
+Wire Wire Line
+	7200 1300 7200 1200
+Connection ~ 7200 1400
+Wire Wire Line
+	7200 1400 7200 1300
+Connection ~ 7200 1500
+Wire Wire Line
+	7200 1500 7200 1400
+Connection ~ 7200 1600
+Wire Wire Line
+	7200 1600 7200 1500
+Connection ~ 7200 1700
+Wire Wire Line
+	7200 1700 7200 1600
+Connection ~ 7200 1800
+Wire Wire Line
+	7200 1800 7200 1700
 $EndSCHEMATC

Commit message: Finish initial layout
Parts:
- removed J3: Conn_02x10_Odd_Even, Connector_PinHeader_1.27mm:PinHeader_2x10_P1.27mm_Vertical, symbol Connector_Generic:Conn_02x10_Odd_Even
- removed SW1, SW2, SW3: SW_Push_Dual, Button_Switch_SMD:SW_SPST_EVPBF, symbol Switch:SW_Push_Dual
- added J14, J15, J19: Conn_01x02_Male, Connector_PinHeader_2.54mm:PinHeader_1x02_P2.54mm_Vertical, symbol Connector:Conn_01x02_Male
- added J3: Conn_02x05_Odd_Even, Connector_PinHeader_1.27mm:PinHeader_2x05_P1.27mm_Vertical, symbol Connector_Generic:Conn_02x05_Odd_Even
Connections:
- net +3V3: now also J14.2 (Pin_2), J15.2 (Pin_2), J3.1 (Pin_1)
- net BOOT0: now also J14.1 (Pin_1)
- net GND: now also J19.1 (Pin_1), J3.3 (Pin_3), J3.5 (Pin_5), J3.9 (Pin_9)
- net NRST: now also J19.2 (Pin_2), J3.10 (Pin_10)
- net RA8875_INT: now also U3.38 (PC7); no longer U3.26 (PB0)
- net RA8875_NRST: now also U3.41 (PA8); no longer U3.39 (PC8)
- net RA8875_WAIT: now also U3.37 (PC6); no longer U3.27 (PB1)
- net SPI_INT: now also U3.28 (PB2); no longer U3.41 (PA8)
- net SWCLK: now also J3.4 (Pin_4)
- net SWDIO: now also J3.2 (Pin_2)
- net USR_PUSHBTN: now also J15.1 (Pin_1)
- no-connect marks 41 -> 38
Changed lines of the file:
@@
 Wire Wire Line
 	2650 5800 2750 5800
-Wire Wire Line
-	1300 5100 1450 5100
 Text Notes 7900 2150 0    50   ~ 0
 RA8875 Connector
@@
 L power:GND #PWR028
 U 1 1 6102234A
-P 7250 1950
-F 0 "#PWR028" H 7250 1700 50  0001 C CNN
-F 1 "GND" H 7100 1900 50  0000 C CNN
-F 2 "" H 7250 1950 50  0001 C CNN
-F 3 "" H 7250 1950 50  0001 C CNN
-	1    7250 1950
+P 6650 1450
+F 0 "#PWR028" H 6650 1200 50  0001 C CNN
+F 1 "GND" H 6500 1400 50  0000 C CNN
+F 2 "" H 6650 1450 50  0001 C CNN
+F 3 "" H 6650 1450 50  0001 C CNN
+	1    6650 1450
 	1    0    0    -1
 $EndComp
@@
 Wire Wire Line
 	1300 2600 1450 2600
-Text Label 6700 1700 2    50   ~ 0
+Text Label 7200 1400 0    50   ~ 0
 NRST
-Text Label 6700 1300 2    50   ~ 0
+Text Label 7200 1000 0    50   ~ 0
 SWDIO
-Text Label 6700 1400 2    50   ~ 0
+Text Label 7200 1100 0    50   ~ 0
 SWCLK
 $Comp
@@
 Text Label 5900 3700 2    50   ~ 0
 NRST
-Wire Wire Line
-	5900 3700 5900 3800
 $Comp
 L power:GND #PWR024
@@
 	0    1    1    0
 $EndComp
-Wire Wire Line
-	5900 3800 6000 3800
-Connection ~ 5900 3800
 Wire Wire Line
 	6350 3800 6350 3700
@@
 	5650 4100 5650 4200
 Wire Wire Line
-	5650 4200 5800 4200
-Wire Wire Line
 	5650 3900 5650 3800
-Wire Wire Line
-	5650 3800 5800 3800
 Text Label 2800 3500 0    50   ~ 0
 USART_TX
@@
 Reset/Boot Circuitry
 Wire Notes Line
-	7450 1650 7450 700
-Wire Notes Line
 	7450 700  6400 700
-Wire Notes Line
-	6400 700  6400 1650
 Text Notes 6400 700  0    50   ~ 0
 Debug Connector\n
@@
 NoConn ~ 2650 3800
 NoConn ~ 2650 4100
-NoConn ~ 2650 4500
+NoConn ~ 2650 4400
 NoConn ~ 2650 4600
 NoConn ~ 2650 4700
@@
 NoConn ~ 1450 5300
 NoConn ~ 1450 5200
-NoConn ~ 1450 5000
-NoConn ~ 1450 4900
+NoConn ~ 2650 4300
+NoConn ~ 1450 5100
 NoConn ~ 1450 4800
 NoConn ~ 1450 4700
@@
 NoConn ~ 1450 3700
 NoConn ~ 1450 3600
-Wire Wire Line
-	2800 4400 2650 4400
-Wire Wire Line
-	2650 4300 2800 4300
 Text Label 8050 2900 0    50   ~ 0
 RA8875_WAIT
@@
 Wire Wire Line
 	7800 4650 7850 4650
-Text Label 2800 3400 0    50   ~ 0
+Text Label 2800 4500 0    50   ~ 0
 SUBS_P_INT
 Wire Wire Line
-	2650 3400 2800 3400
+	2650 4500 2800 4500
 $Comp
 L Connector:Conn_01x05_Male J5
@@
 Wire Wire Line
 	7050 4950 7100 4950
-Text Label 1300 5100 2    50   ~ 0
+Text Label 2650 3400 0    50   ~ 0
 RA8875_NRST
 Text Label 2750 5500 0    50   ~ 0
@@
 Text Label 2750 5600 0    50   ~ 0
 RA8875_SCK
-Text Label 2800 4300 0    50   ~ 0
+Text Label 1450 5000 2    50   ~ 0
 RA8875_INT
-Text Label 2800 4400 0    50   ~ 0
+Text Label 1450 4900 2    50   ~ 0
 RA8875_WAIT
 $Comp
@@
 Wire Notes Line
 	6550 5300 10350 5300
-$Comp
-L Switch:SW_Push_Dual SW2
-U 1 1 60A9B835
-P 6050 2700
-F 0 "SW2" H 5900 2800 50  0000 L CNN
-F 1 "SW_Push_Dual" H 5700 2900 50  0000 L CNN
-F 2 "Button_Switch_SMD:SW_SPST_EVPBF" H 6050 2900 50  0001 C CNN
-F 3 "~" H 6050 2900 50  0001 C CNN
-F 4 "Pushbuttons for NRST/BOOT" H 6050 2700 50  0001 C CNN "Description"
-	1    6050 2700
-	0    1    1    0
-$EndComp
 Wire Wire Line
 	5700 3250 5700 3200
 Wire Wire Line
-	6050 2950 6050 2900
-Wire Wire Line
 	5700 2950 5700 3000
-Wire Wire Line
-	5850 2950 5850 2900
 $Comp
 L power:+3.3V #PWR025
@@
 Wire Wire Line
 	6050 2450 6050 2500
-Wire Wire Line
-	6050 2500 5850 2500
-Connection ~ 6050 2500
 $Comp
 L Device:C_Small C9
@@
 $EndComp
 Wire Wire Line
-	5850 2950 5700 2950
-Wire Wire Line
 	5700 2950 5700 2800
-Connection ~ 5850 2950
 Wire Wire Line
 	5700 2600 5700 2500
-Wire Wire Line
-	5700 2500 5850 2500
-Connection ~ 5850 2500
-$Comp
-L Switch:SW_Push_Dual SW1
-U 1 1 60BBAAA3
-P 6000 4000
-F 0 "SW1" H 6000 4100 50  0000 L CNN
-F 1 "SW_Push_Dual" H 5850 4200 50  0000 L CNN
-F 2 "Button_Switch_SMD:SW_SPST_EVPBF" H 6000 4200 50  0001 C CNN
-F 3 "~" H 6000 4200 50  0001 C CNN
-F 4 "Pushbuttons for NRST/BOOT" H 6000 4000 50  0001 C CNN "Description"
-	1    6000 4000
-	0    1    1    0
-$EndComp
-Connection ~ 6000 3800
-Connection ~ 5800 3800
-Wire Wire Line
-	5800 3800 5900 3800
-Connection ~ 5800 4200
-Wire Wire Line
-	5800 4200 5900 4200
-Connection ~ 5900 4200
-Wire Wire Line
-	5900 4200 6000 4200
 Connection ~ 5700 2950
 Wire Wire Line
-	5850 2950 6050 2950
-Wire Wire Line
 	6150 3000 6150 2950
-Wire Wire Line
-	6150 2950 6050 2950
-Connection ~ 6050 2950
-Wire Wire Line
-	6000 3800 6100 3800
 Wire Wire Line
 	6300 3800 6350 3800
@@
 Wire Notes Line
 	7850 4050 7850 3250
-$Comp
-L Switch:SW_Push_Dual SW3
-U 1 1 60FDEA1B
-P 6100 1200
-F 0 "SW3" H 6100 1300 50  0000 L CNN
-F 1 "SW_Push_Dual" H 5800 1400 50  0000 L CNN
-F 2 "Button_Switch_SMD:SW_SPST_EVPBF" H 6100 1400 50  0001 C CNN
-F 3 "~" H 6100 1400 50  0001 C CNN
-F 4 "User push button" H 6100 1200 50  0001 C CNN "Description"
-	1    6100 1200
-	0    1    1    0
-$EndComp
 Text Label 5650 1400 3    50   ~ 0
 USR_PUSHBTN
@@
 	5900 1700 5900 1650
 Wire Wire Line
-	6100 1400 5900 1400
-Wire Wire Line
 	5650 1000 5900 1000
 Connection ~ 5900 1000
 Wire Wire Line
-	5900 1000 6100 1000
+	5900 1000 5950 1000
 $Comp
 L power:+3.3V #PWR022
@@
 Wire Wire Line
 	9450 2600 10050 2600
-$Comp
-L Connector_Generic:Conn_02x10_Odd_Even J3
-U 1 1 606691DA
-P 6900 1400
-F 0 "J3" H 6950 2017 50  0000 C CNN
-F 1 "Conn_02x10_Odd_Even" V 7300 1350 50  0000 C CNN
-F 2 "Connector_PinHeader_1.27mm:PinHeader_2x10_P1.27mm_Vertical" H 6900 1400 50  0001 C CNN
-F 3 "~" H 6900 1400 50  0001 C CNN
-	1    6900 1400
-	1    0    0    -1
-$EndComp
-NoConn ~ 6700 1500
-NoConn ~ 6700 1600
-NoConn ~ 6700 1800
-NoConn ~ 6700 1900
-NoConn ~ 6700 1100
-NoConn ~ 6700 1200
 Wire Wire Line
 	6650 950  6650 1000
 Wire Wire Line
 	6650 1000 6700 1000
-Wire Wire Line
-	7250 1950 7250 1900
-Wire Wire Line
-	7250 1900 7200 1900
-Wire Wire Line
-	7200 1900 7200 1800
-Connection ~ 7200 1900
-Connection ~ 7200 1100
-Wire Wire Line
-	7200 1100 7200 1000
-Connection ~ 7200 1200
-Wire Wire Line
-	7200 1200 7200 1100
-Connection ~ 7200 1300
-Wire Wire Line
-	7200 1300 7200 1200
-Connection ~ 7200 1400
-Wire Wire Line
-	7200 1400 7200 1300
-Connection ~ 7200 1500
-Wire Wire Line
-	7200 1500 7200 1400
-Connection ~ 7200 1600
-Wire Wire Line
-	7200 1600 7200 1500
-Connection ~ 7200 1700
-Wire Wire Line
-	7200 1700 7200 1600
-Connection ~ 7200 1800
-Wire Wire Line
-	7200 1800 7200 1700
+$Comp
+L Connector_Generic:Conn_02x05_Odd_Even J3
+U 1 1 607A450C
+P 6900 1200
+F 0 "J3" H 6950 1617 50  0000 C CNN
+F 1 "Conn_02x05_Odd_Even" H 6950 1526 50  0000 C CNN
+F 2 "Connector_PinHeader_1.27mm:PinHeader_2x05_P1.27mm_Vertical" H 6900 1200 50  0001 C CNN
+F 3 "~" H 6900 1200 50  0001 C CNN
+	1    6900 1200
+	1    0    0    -1
+$EndComp
+NoConn ~ 7200 1200
+NoConn ~ 7200 1300
+NoConn ~ 6700 1300
+Wire Wire Line
+	6700 1100 6650 1100
+Wire Wire Line
+	6650 1100 6650 1200
+Wire Wire Line
+	6700 1400 6650 1400
+Connection ~ 6650 1400
+Wire Wire Line
+	6650 1400 6650 1450
+Wire Wire Line
+	6700 1200 6650 1200
+Connection ~ 6650 1200
+Wire Wire Line
+	6650 1200 6650 1400
+Wire Notes Line
+	7450 2050 6400 2050
+Wire Notes Line
+	7450 700  7450 2050
+Wire Notes Line
+	6400 700  6400 2050
+Wire Wire Line
+	5650 3800 5850 3800
+Wire Wire Line
+	5650 4200 5850 4200
+$Comp
+L Connector:Conn_01x02_Male J14
+U 1 1 605F435C
+P 6100 2750
+F 0 "J14" H 6072 2632 50  0000 R CNN
+F 1 "Conn_01x02_Male" V 5950 3200 50  0000 R CNN
+F 2 "Connector_PinHeader_2.54mm:PinHeader_1x02_P2.54mm_Vertical" H 6100 2750 50  0001 C CNN
+F 3 "~" H 6100 2750 50  0001 C CNN
+	1    6100 2750
+	-1   0    0    1
+$EndComp
+Wire Wire Line
+	5850 4050 5850 4200
+Connection ~ 5850 4200
+Wire Wire Line
+	5850 4200 5900 4200
+Wire Wire Line
+	5850 3950 5850 3800
+Connection ~ 5850 3800
+Wire Wire Line
+	5700 2500 5900 2500
+Wire Wire Line
+	5700 2950 5900 2950
+Wire Wire Line
+	5900 2650 5900 2500
+Connection ~ 5900 2500
+Wire Wire Line
+	5900 2500 6050 2500
+Wire Wire Line
+	5900 2750 5900 2950
+Connection ~ 5900 2950
+$Comp
+L Connector:Conn_01x02_Male J15
+U 1 1 60625B17
+P 6150 1250
+F 0 "J15" H 6122 1132 50  0000 R CNN
+F 1 "Conn_01x02_Male" V 6000 1700 50  0000 R CNN
+F 2 "Connector_PinHeader_2.54mm:PinHeader_1x02_P2.54mm_Vertical" H 6150 1250 50  0001 C CNN
+F 3 "~" H 6150 1250 50  0001 C CNN
+	1    6150 1250
+	-1   0    0    1
+$EndComp
+Wire Wire Line
+	5950 1150 5950 1000
+Wire Wire Line
+	5950 1250 5950 1400
+Wire Wire Line
+	5950 1400 5900 1400
+Wire Wire Line
+	5900 2950 6150 2950
+Wire Wire Line
+	5850 3800 5900 3800
+Wire Wire Line
+	5900 3800 5900 3700
+Connection ~ 5900 3800
+Wire Wire Line
+	5900 3800 6100 3800
+$Comp
+L Connector:Conn_01x02_Male J19
+U 1 1 606F3729
+P 6050 4050
+F 0 "J19" H 6022 3932 50  0000 R CNN
+F 1 "Conn_01x02_Male" V 5900 4500 50  0000 R CNN
+F 2 "Connector_PinHeader_2.54mm:PinHeader_1x02_P2.54mm_Vertical" H 6050 4050 50  0001 C CNN
+F 3 "~" H 6050 4050 50  0001 C CNN
+	1    6050 4050
+	-1   0    0    1
+$EndComp
 $EndSCHEMATC

Commit message: PCB changes
Parts:
- U3: Digi-Key_PN (none) -> STM32F051R8T6
- U4: Digi-Key_PN (none) -> CAT24C256YI-GT3
- Y1: Digi-Key_PN (none) -> ASDDV-8.000MHZ-LR-T
Changed lines of the file:
@@
 F 3 "http://www.st.com/st-web-ui/static/active/en/resource/technical/document/datasheet/DM00039193.pdf" H 2050 4200 50  0001 C CNN
 F 4 "F0 processor for User IO" H 2050 4200 50  0001 C CNN "Description"
+F 5 "STM32F051R8T6" H 2050 4200 50  0001 C CNN "Digi-Key_PN"
 	1    2050 4200
 	1    0    0    -1
@@
 F 3 "https://www.onsemi.cn/PowerSolutions/document/CAT24C256-D.PDF" H 8100 1400 50  0001 C CNN
 F 4 "EEPROM for storage" H 8100 1400 50  0001 C CNN "Description"
+F 5 "CAT24C256YI-GT3" H 8100 1400 50  0001 C CNN "Digi-Key_PN"
 	1    8100 1400
 	1    0    0    -1
@@
 F 3 "~" H 7100 3500 50  0001 C CNN
 F 4 "HSE crystals" H 7100 3500 50  0001 C CNN "Description"
+F 5 "ASDDV-8.000MHZ-LR-T" H 7100 3500 50  0001 C CNN "Digi-Key_PN"
 	1    7100 3500
 	1    0    0    -1
