File: user_io.sch (KiCad schematic (older format))
At the start: 39 parts, among them J14 Conn_01x02_Male, J15 Conn_01x02_Male, J19 Conn_01x02_Male, J3 Conn_02x05_Odd_Even, J4 Conn_01x06_Male, J5 Conn_01x05_Male, J6 Conn_01x04_Male, J7 Conn_01x09_Male, J8 Conn_01x04_Male, U3 STM32F051R8T6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

Commit message: Updated
Parts:
- J3: footprint Connector_PinHeader_1.27mm:PinHeader_2x05_P1.27mm_Vertical -> Connector_PinHeader_1.27mm:PinHeader_2x05_P1.27mm_Vertical_SMD
Changed lines of the file:
@@
 F 0 "J3" H 6950 1617 50  0000 C CNN
 F 1 "Conn_02x05_Odd_Even" H 6950 1526 50  0000 C CNN
-F 2 "Connector_PinHeader_1.27mm:PinHeader_2x05_P1.27mm_Vertical" H 6900 1200 50  0001 C CNN
+F 2 "Connector_PinHeader_1.27mm:PinHeader_2x05_P1.27mm_Vertical_SMD" H 6900 1200 50  0001 C CNN
 F 3 "~" H 6900 1200 50  0001 C CNN
 	1    6900 1200
